File: XpressoSmoothie.sch (KiCad schematic (older format))
At the start: 51 parts

Commit message: Added power plug and first mosfet.
Parts:
- removed J?: HEADER_4, symbol HEADER_4
- added C?: 100u, symbol CP1
- added C?: 100n, symbol C
- added D? (x2): LED, symbol LED
- added D?: 1N4004, symbol DIODE
- added F? (x2): FUSE, symbol FUSE
- added J?: HEADER_4, symbol HEADER_4
- added J?: HEADER_2, symbol HEADER_2
- added Q?: IRLB 8743, symbol MOSFET_N_RMC
- added Q?: 2N7000K, symbol MOS_N
- added R?: R, symbol R
- added R?: 10R, symbol R
- added R?: 10K, symbol R
- added R?: 1K8, symbol R
Connections:
- net labels added: +12P, LED, POWER1
- wire segments 278 -> 316
Other:
- moved on the sheet: C?

Commit message: Finish wiring labels.
Parts:
- added D? (x3): LED, symbol LED
- added J? (x3): HEADER_2, symbol HEADER_2
- added Q? (x3): 2N7000K, symbol MOS_N
- added Q? (x3): IRLB 8743, symbol MOSFET_N_RMC
- added R? (x3): 1K8, symbol R
- added R? (x3): 10K, symbol R
- added R? (x3): 10R, symbol R
Connections:
- net labels added: POWER2, POWER3, POWER4
- wire segments 316 -> 399
Other:
- moved on the sheet: D?, J?, Q?, R?

Commit message: Switch around pins and add pins for UART. Finish most of netlist.
Parts:
- removed C? (x5): 100u, symbol C
- added C1, C12, C2, C3, C4: 100u, symbol CP1
- added J15: HEADER_2, symbol HEADER_2
- C5, C6: renamed from C?; value C -> 100n
- D1: renamed from D?; value LED -> LED_GREEN
- D3, D4, D5, D6: renamed from D?; value LED -> LED_RED
- R7: renamed from R?; value R -> 1k
- gave numbers to parts that had none: 73
Connections:
- net labels added: RX, TX
- wire segments 399 -> 403

Commit message: Minor tag issues.
Parts:
- removed J6: LPCXpresso_1769_Header, symbol LPCXpresso_1769_Header
- added J6: LPCXPRESSO_GENERIC_HEADER, symbol LPCXPRESSO_GENERIC_HEADER

Commit message: Add screw terminal .mod file, plus tons of fixes/layout changes.
Parts:
- removed J15: HEADER_2, symbol HEADER_2
- removed JP1: USB-B, symbol USB-B
- added J26: USB_1, symbol USB_1
Connections:
- net labels removed: RX, TX

Commit message: Everything placed approximately.
Connections:
- wire segments 403 -> 405
Other:
- moved on the sheet: D2
Changed lines of the file:
@@
-EESchema Schematic File Version 2  date Tue 14 May 2013 02:01:36 PM EDT
+EESchema Schematic File Version 2  date Tue 14 May 2013 02:47:57 PM EDT
 LIBS:power
 LIBS:device
@@
 Comment4 ""
 $EndDescr
+Connection ~ 6600 3100
+Wire Wire Line
+	6600 3100 6600 3050
+Wire Wire Line
+	6350 3200 6500 3200
+Wire Wire Line
+	6350 3200 6350 3500
+Wire Wire Line
+	6350 3500 6050 3500
 Wire Wire Line
 	700  2300 900  2300
@@
 Connection ~ 3900 4500
 Wire Wire Line
-	3900 4400 3900 4600
+	3900 4600 3900 4400
 Wire Wire Line
 	3900 4400 4000 4400
 Wire Wire Line
-	3850 4600 3850 4650
+	3850 4650 3850 4600
 Wire Wire Line
 	3850 4600 4750 4600
@@
 	4050 5800 3900 5800
 Wire Wire Line
-	3900 5250 3900 5800
-Wire Wire Line
-	2900 5250 3900 5250
+	3900 5800 3900 5250
+Wire Wire Line
+	3900 5250 2900 5250
 Connection ~ 3750 5900
 Wire Wire Line
@@
 Connection ~ 6900 3600
 Wire Wire Line
-	7300 3600 7300 3550
-Wire Wire Line
-	6500 3600 7300 3600
-Wire Wire Line
-	6100 3600 5100 3600
+	7300 3550 7300 3600
 Wire Wire Line
 	5100 3300 5550 3300
@@
 Connection ~ 2800 3550
 Wire Wire Line
-	2800 3350 2900 3350
-Wire Wire Line
-	2800 4300 2800 3350
+	2900 3350 2800 3350
+Wire Wire Line
+	2800 3350 2800 4300
 Connection ~ 2800 4200
 Wire Wire Line
@@
 	1250 3150 1400 3150
 Wire Wire Line
-	1250 3550 1400 3550
+	1400 3550 1250 3550
 Connection ~ 2200 3450
 Wire Wire Line
@@
 Connection ~ 5600 1300
 Wire Wire Line
-	5450 1300 5450 1600
-Wire Wire Line
-	5750 1300 5450 1300
+	5450 1600 5450 1300
+Wire Wire Line
+	5450 1300 5750 1300
 Wire Wire Line
 	7100 1550 7600 1550
@@
 	7500 1100 7400 1100
 Wire Wire Line
-	7500 1300 7400 1300
+	7400 1300 7500 1300
 Connection ~ 7050 1300
 Wire Wire Line
-	7050 1650 7050 1300
+	7050 1300 7050 1650
 Wire Wire Line
 	7050 1650 6700 1650
@@
 Connection ~ 7500 1200
 Wire Wire Line
-	7500 800  7500 1300
+	7500 1300 7500 800
 Wire Wire Line
 	6950 900  7500 900
@@
 Connection ~ 8150 1450
 Wire Wire Line
-	8150 1650 8150 1450
+	8150 1450 8150 1650
 Wire Wire Line
 	8150 1650 8300 1650
@@
 	10500 1750 10500 1600
 Wire Wire Line
-	10850 1600 10850 1450
+	10850 1450 10850 1600
 Wire Wire Line
 	10300 850  10200 850
@@
 	10650 1250 10750 1250
 Wire Wire Line
-	10350 1600 10350 1450
+	10350 1450 10350 1600
 Wire Wire Line
 	10350 1450 10200 1450
@@
 Connection ~ 10750 900
 Wire Wire Line
-	10850 1600 10350 1600
+	10350 1600 10850 1600
 Wire Wire Line
 	9000 1350 8700 1350
@@
 Connection ~ 8850 1350
 Wire Wire Line
-	7950 1450 7950 1200
-Wire Wire Line
-	9000 1450 7950 1450
+	7950 1200 7950 1450
+Wire Wire Line
+	7950 1450 9000 1450
 Connection ~ 4900 2600
 Wire Wire Line
-	4900 2800 4900 2600
+	4900 2600 4900 2800
 Wire Wire Line
 	4900 2800 5050 2800
@@
 	7250 2900 7250 2750
 Wire Wire Line
-	7600 2750 7600 2600
+	7600 2600 7600 2750
 Wire Wire Line
 	7050 2000 6950 2000
@@
 	7400 2400 7500 2400
 Wire Wire Line
-	7100 2750 7100 2600
+	7100 2600 7100 2750
 Wire Wire Line
 	7100 2600 6950 2600
@@
 Connection ~ 7500 2050
 Wire Wire Line
-	7600 2750 7100 2750
+	7100 2750 7600 2750
 Wire Wire Line
 	5750 2500 5450 2500
@@
 Connection ~ 5600 2500
 Wire Wire Line
-	4700 2600 4700 2350
-Wire Wire Line
-	5750 2600 4700 2600
+	4700 2350 4700 2600
+Wire Wire Line
+	4700 2600 5750 2600
 Wire Wire Line
 	9050 2600 8000 2600
@@
 Connection ~ 8900 2500
 Wire Wire Line
-	8750 2500 8750 2800
-Wire Wire Line
-	9050 2500 8750 2500
+	8750 2800 8750 2500
+Wire Wire Line
+	8750 2500 9050 2500
 Wire Wire Line
 	10400 2750 10900 2750
@@
 	10800 2300 10700 2300
 Wire Wire Line
-	10800 2500 10700 2500
+	10700 2500 10800 2500
 Connection ~ 10350 2500
 Wire Wire Line
-	10350 2850 10350 2500
+	10350 2500 10350 2850
 Wire Wire Line
 	10350 2850 10000 2850
@@
 Connection ~ 10800 2400
 Wire Wire Line
-	10800 2000 10800 2500
+	10800 2500 10800 2000
 Wire Wire Line
 	10250 2100 10800 2100
@@
 Connection ~ 8250 3800
 Wire Wire Line
-	8250 4000 8250 3800
+	8250 3800 8250 4000
 Wire Wire Line
 	8250 4000 8400 4000
@@
 	10600 4100 10600 3950
 Wire Wire Line
-	10950 3950 10950 3800
+	10950 3800 10950 3950
 Wire Wire Line
 	10400 3200 10300 3200
@@
 	10750 3600 10850 3600
 Wire Wire Line
-	10450 3950 10450 3800
+	10450 3800 10450 3950
 Wire Wire Line
 	10450 3800 10300 3800
@@
 Connection ~ 10850 3250
 Wire Wire Line
-	10950 3950 10450 3950
+	10450 3950 10950 3950
 Wire Wire Line
 	9100 3700 8800 3700
@@
 Connection ~ 8950 3700
 Wire Wire Line
-	8050 3800 8050 3550
-Wire Wire Line
-	9100 3800 8050 3800
+	8050 3550 8050 3800
+Wire Wire Line
+	8050 3800 9100 3800
 Wire Wire Line
 	800  1000 800  800
@@
 Connection ~ 2200 3250
 Wire Wire Line
-	1250 3050 1250 3550
+	1250 3550 1250 3050
 Wire Wire Line
 	1400 3350 1250 3350
@@
 Connection ~ 2400 3450
 Wire Wire Line
-	2150 4200 2150 4100
-Wire Wire Line
-	2800 4200 2150 4200
+	2150 4100 2150 4200
+Wire Wire Line
+	2150 4200 2800 4200
 Wire Wire Line
 	2400 4100 2400 4200
@@
 	5100 3500 5550 3500
 Wire Wire Line
-	6050 3500 6600 3500
-Wire Wire Line
-	6600 3100 6600 3600
-Connection ~ 6600 3500
-Wire Wire Line
 	6900 3600 6900 3550
-Connection ~ 6600 3600
-Wire Wire Line
-	7300 3100 7300 3150
-Wire Wire Line
-	6600 3100 7300 3100
+Wire Wire Line
+	7300 3150 7300 3100
 Wire Wire Line
 	6050 3300 6300 3300
@@
 	6300 3300 6300 3100
 Wire Wire Line
-	2900 6950 2900 6800
+	2900 6800 2900 6950
 Wire Wire Line
 	2900 6950 3750 6950
@@
 	3450 5450 3600 5450
 Wire Wire Line
-	2900 5700 2900 5250
+	2900 5250 2900 5700
 Wire Wire Line
 	3100 5250 3100 5150
@@
 	5150 5100 5150 5200
 Wire Wire Line
-	4950 5200 4950 5650
+	4950 5650 4950 5200
 Wire Wire Line
 	5500 5400 5650 5400
@@
 	4950 6150 4950 6350
 Wire Wire Line
-	5800 6900 5800 6400
+	5800 6400 5800 6900
 Wire Wire Line
 	5800 6900 4950 6900
@@
 	4950 5400 5000 5400
 Wire Wire Line
-	5650 5850 5650 5800
-Wire Wire Line
-	6100 5850 5650 5850
+	5650 5800 5650 5850
+Wire Wire Line
+	5650 5850 6100 5850
 Connection ~ 5800 5850
 Wire Wire Line
@@
 	8350 5350 8200 5350
 Wire Wire Line
-	8200 4800 8200 5350
-Wire Wire Line
-	7200 4800 8200 4800
+	8200 5350 8200 4800
+Wire Wire Line
+	8200 4800 7200 4800
 Connection ~ 8050 5450
 Wire Wire Line
@@
 	7750 5850 7200 5850
 Wire Wire Line
-	7200 6500 7200 6350
+	7200 6350 7200 6500
 Wire Wire Line
 	7200 6500 8050 6500
@@
 	7750 5000 7900 5000
 Wire Wire Line
-	7200 5250 7200 4800
+	7200 4800 7200 5250
 Wire Wire Line
 	7400 4800 7400 4700
@@
 	9800 4800 9800 4900
 Wire Wire Line
-	9600 4900 9600 5350
+	9600 5350 9600 4900
 Wire Wire Line
 	10150 5100 10300 5100
@@
 	9600 5850 9600 6050
 Wire Wire Line
-	10450 6600 10450 6100
+	10450 6100 10450 6600
 Wire Wire Line
 	10450 6600 9600 6600
@@
 	9600 5100 9650 5100
 Wire Wire Line
-	10300 5550 10300 5500
-Wire Wire Line
-	10750 5550 10300 5550
+	10300 5500 10300 5550
+Wire Wire Line
+	10300 5550 10750 5550
 Connection ~ 10450 5550
 Wire Wire Line
@@
 Wire Wire Line
 	850  2250 700  2250
+Wire Wire Line
+	7300 3600 5100 3600
+Connection ~ 6500 3600
+Wire Wire Line
+	6500 3200 6500 3100
+Wire Wire Line
+	6500 3100 7300 3100
 $Comp
 L GND #PWR01
@@
 L DIODE D2
 U 1 1 51900DA8
-P 6300 3600
-F 0 "D2" H 6300 3700 40  0000 C CNN
-F 1 "1N4004" H 6300 3500 40  0000 C CNN
-	1    6300 3600
-	1    0    0    1
+P 6500 3400
+F 0 "D2" H 6500 3500 40  0000 C CNN
+F 1 "1N4004" H 6500 3300 40  0000 C CNN
+	1    6500 3400
+	0    1    -1   0
 $EndComp
 $Comp
@@
 L +12V #PWR012
 U 1 1 51900CFB
-P 6600 3100
-F 0 "#PWR012" H 6600 3050 20  0001 C CNN
-F 1 "+12V" H 6600 3200 30  0000 C CNN
-	1    6600 3100
-	1    0    0    -1
-$EndComp
+P 6600 3050
+F 0 "#PWR012" H 6600 3000 20  0001 C CNN
+F 1 "+12V" H 6600 3150 30  0000 C CNN
+	1    6600 3050
+	1    0    0    -1
+$EndComp

Commit message: Switch out header for proper SD card connector.
Parts:
- removed J3: HEADER_7, symbol HEADER_7
- added R27, R28, R29: 10k, symbol R
- added U6: CONN_MICROSD, symbol CONN_MICROSD
Connections:
- net labels removed: CD
- wire segments 405 -> 415

Commit message: Begun laying traces.
Connections:
- wire segments 415 -> 414
Other:
- moved on the sheet: J13
Changed lines of the file:
@@
-EESchema Schematic File Version 2  date Tue 14 May 2013 03:20:14 PM EDT
+EESchema Schematic File Version 2  date Tue 14 May 2013 05:12:31 PM EDT
 LIBS:power
 LIBS:device
@@
 Comment4 ""
 $EndDescr
+Connection ~ 2800 3550
+Wire Wire Line
+	2900 3550 2800 3550
+Wire Wire Line
+	2900 3150 2800 3150
+Wire Wire Line
+	2800 3150 2800 4300
+Wire Wire Line
+	2900 3450 2050 3450
+Connection ~ 2650 3250
+Wire Wire Line
+	700  2200 900  2200
+Wire Wire Line
+	700  2300 900  2300
 Connection ~ 2650 850
 Wire Wire Line
@@
 	5100 3600 7300 3600
 Wire Wire Line
-	850  2250 700  2250
-Wire Wire Line
 	2350 2200 2100 2200
 Wire Wire Line
@@
 	2150 1650 2350 1650
 Wire Wire Line
-	900  1550 700  1550
-Wire Wire Line
 	2350 1450 2150 1450
 Wire Wire Line
@@
 Wire Wire Line
 	750  1650 900  1650
-Connection ~ 2800 3750
-Wire Wire Line
-	2800 3550 2900 3550
 Connection ~ 2400 4200
 Wire Wire Line
@@
 Wire Wire Line
 	2200 3550 1900 3550
-Wire Wire Line
-	2900 3450 2050 3450
 Wire Wire Line
 	2250 2300 2100 2300
@@
 	4050 1850 4050 2450
 Wire Wire Line
-	2050 3650 2900 3650
-Wire Wire Line
-	2700 3250 2900 3250
-Wire Wire Line
 	1900 3350 2200 3350
 Wire Wire Line
@@
 Connection ~ 2150 3650
 Wire Wire Line
-	2650 3700 2650 3250
-Wire Wire Line
-	2650 3250 2050 3250
-Connection ~ 2700 3250
+	2650 3250 2650 3700
 Wire Wire Line
 	2650 4200 2650 4100
 Connection ~ 2650 4200
-Wire Wire Line
-	2800 3750 2900 3750
 Connection ~ 2800 4200
-Wire Wire Line
-	2800 4300 2800 3350
-Wire Wire Line
-	2800 3350 2900 3350
-Connection ~ 2800 3550
 Wire Wire Line
 	850  1700 750  1700
@@
 	2100 1500 2350 1500
 Wire Wire Line
-	700  1500 850  1500
-Wire Wire Line
 	4750 4250 4850 4250
 Wire Wire Line
@@
 	2350 2150 2150 2150
 Wire Wire Line
-	700  2200 900  2200
-Wire Wire Line
-	700  2300 900  2300
-Wire Wire Line
 	6050 3500 6350 3500
 Wire Wire Line
@@
 	3450 850  3450 950
 Connection ~ 3450 950
+Wire Wire Line
+	2350 2250 2150 2250
+Wire Wire Line
+	850  2350 700  2350
+Wire Wire Line
+	850  2250 700  2250
+Wire Wire Line
+	2900 3250 2050 3250
+Wire Wire Line
+	2900 3650 2050 3650
+Wire Wire Line
+	2900 3350 2800 3350
+Connection ~ 2800 3350
 $Comp
 L R R29
@@
 Text GLabel 700  1800 0    30   Input ~ 0
 XMAX
-Text GLabel 700  2200 0    30   Input ~ 0
+Text GLabel 2350 2250 2    30   Input ~ 0
 B-EN
-Text GLabel 700  2250 0    30   Input ~ 0
+Text GLabel 700  2300 0    30   Input ~ 0
 B-STEP
-Text GLabel 700  2300 0    30   Input ~ 0
+Text GLabel 700  2350 0    30   Input ~ 0
 B-DIR
-Text GLabel 2350 2100 2    30   Input ~ 0
+Text GLabel 2350 2200 2    30   Input ~ 0
 A-DIR
 Text GLabel 2350 2150 2    30   Input ~ 0
 A-STEP
-Text GLabel 2350 2200 2    30   Input ~ 0
+Text GLabel 2350 2100 2    30   Input ~ 0
 A-EN
 Text GLabel 2350 1850 2    30   Input ~ 0
@@
 Text GLabel 700  1450 0    30   Input ~ 0
 POWER3
-Text GLabel 700  1500 0    30   Input ~ 0
+Text GLabel 700  2200 0    30   Input ~ 0
 POWER2
-Text GLabel 700  1550 0    30   Input ~ 0
+Text GLabel 700  2250 0    30   Input ~ 0
 POWER1
 $Comp
@@
 	1    0    0    -1
 $EndComp
-Text GLabel 2050 3650 0    30   Input ~ 0
+Text GLabel 2050 3250 0    30   Input ~ 0
 THERM2
 Text GLabel 2050 3450 0    30   Input ~ 0
 THERM1
-Text GLabel 2050 3250 0    30   Input ~ 0
+Text GLabel 2050 3650 0    30   Input ~ 0
 THERM0
 $Comp
@@
 L HEADER_6 J13
 U 1 1 518FFBEF
-P 3000 3500
-F 0 "J13" H 3000 3850 60  0000 C CNN
-F 1 "HEADER_6" H 3000 3150 60  0000 C CNN
-	1    3000 3500
-	1    0    0    -1
-$EndComp
+P 3000 3400
+F 0 "J13" H 3000 3750 60  0000 C CNN
+F 1 "HEADER_6" H 3000 3050 60  0000 C CNN
+	1    3000 3400
+	1    0    0    -1
+$EndComp
