File: XpressoSmoothie.sch (KiCad schematic (older format))
At the start: 89 parts, among them J1 HEADER_4, J10 HEADER_3X2, J11 HEADER_4, J12 HEADER_4, J13 HEADER_6, J14 HEADER_3X2, J16 HEADER_3, J17 HEADER_3, J18 HEADER_3, J19 HEADER_2, J2 HEADER_4, J20 HEADER_2, J21 HEADER_2, J22 HEADER_2, J23 HEADER_3, J24 HEADER_3, J25 HEADER_3, J26 USB_1, J4 HEADER_3X2, J5 HEADER_3X2, J6 LPCXPRESSO_GENERIC_HEADER, J7 HEADER_4, J8 HEADER_4, J9 HEADER_3X2, Q1 IRLB 8743, Q2 IRLB 8743, Q3 2N7000K, Q4 IRLB 8743, Q5 IRLB 8743, Q6 2N7000K, Q7 2N7000K, Q8 2N7000K, SW1 SW_PUSH, SW2 SW_PUSH, U1 POLOLU_A4988, U2 POLOLU_A4988, U3 POLOLU_A4988, U4 POLOLU_A4988, U5 POLOLU_A4988, U6 CONN_MICROSD

Commit message: Bunch of tracks made. A few minor label issues fixed.
Connections:
- wire segments 414 -> 415

Commit message: Add LM1117 and jumper to power from 12V or from USB.
Parts:
- added 20u (x2): CP1, symbol CP1
- added J?: HEADER_3, symbol HEADER_3
- added U?: LM1117, symbol LM1117
Connections:
- net labels added: VIN
- wire segments 415 -> 428
Other:
- moved on the sheet: D3, D4, D5, D6, J19, J20, J21, J22, J26, Q1, Q2, Q4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

Commit message: Fixed stupid labelling error.
Parts:
- removed 20u (x2): CP1, symbol CP1
- added C13, C14: 20u, symbol CP1
- gave numbers to parts that had none: 2

Commit message: Start making changes suggested by NoobMan.
Parts:
- removed Q8: 2N7000K, symbol MOS_N
- removed R24: 10K, symbol R
- added U?: ZXGD3005E6, SOT26, symbol ZXGD3005E6
- R26: value 10R -> 1k
Connections:
- wire segments 428 -> 432
Other:
- moved on the sheet: D5, D6, J21, J22, Q4, Q5, R17, R18, R23, R25

Commit message: Fixed FETs so that they're non-inverting.
Parts:
- removed D3, D4, D5: LED_RED, symbol LED
- removed J19, J20, J21: HEADER_2, symbol HEADER_2
- removed Q1, Q2, Q4: IRLB 8743, symbol MOSFET_N_RMC
- removed Q3, Q6, Q7: 2N7000K, symbol MOS_N
- removed R15, R16, R17: 1K8, symbol R
- removed R19, R20, R23: 10K, symbol R
- removed R21, R22, R25: 10R, symbol R
- added D? (x3): LED_RED, symbol LED
- added J? (x3): HEADER_2, symbol HEADER_2
- added Q? (x3): IRLB 8743, symbol MOSFET_N_RMC
- added R? (x3): 1K8, symbol R
- added R? (x3): 1k, symbol R
- added U? (x3): ZXGD3005E6, SOT26, symbol ZXGD3005E6
Connections:
- wire segments 432 -> 440
Other:
- moved on the sheet: R26, U?

Commit message: Added I2C header.
Parts:
- added J?: HEADER_4, symbol HEADER_4
- added R? (x2): 4k7, symbol R
Connections:
- net labels added: SCL, SDA
- wire segments 440 -> 450

Commit message: Fixed up netlist and footprints, being layout attempt 2.
Parts:
- gave numbers to parts that had none: 22

Commit message: Started new layout. Let's see how this goes...
Parts:
- removed D2: 1N4004, symbol DIODE
