File: XpressoSmoothie.sch (KiCad schematic (older format))
At the start: 114 parts, among them J1 HEADER_4, J10 HEADER_3X2, J11 Pwr_in, J12 HEADER_4, J13 HEADER_4, J14 HEADER_3X2, J15 HEADER_4, J16 HEADER_3, J17 HEADER_3, J18 HEADER_3, J19 HEADER_2, J2 HEADER_4, J20 HEADER_2, J21 HEADER_2, J22 HEADER_2, J23 HEADER_3, J24 HEADER_3, J25 HEADER_3, J26 USB, J27 HEADER_4, J3 HEADER_3, J4 HEADER_3X2, J5 HEADER_3X2, J6 LPCXPRESSO_GENERIC_HEADER, J7 HEADER_4, J8 HEADER_4, J9 HEADER_3X2, Q1 IRLB 8743, Q2 IRLB 8743, Q3 IRLB 8743, Q4 IRLB 8743, SW1 SW_PUSH, SW2 SW_PUSH, U1 POLOLU_A4988, U10 TC4422A, U11 TC4422A, U12 LM1117-3.3, U2 POLOLU_A4988, U3 POLOLU_A4988, U4 POLOLU_A4988, U5 POLOLU_A4988, U6 CONN_MICROSD, U7 LM7812CT, U8 TC4422A, U9 TC4422A

Commit message: spaced the 4 pololu on top
spaced the 4 pololu on top
Other:
- note added: "Capacitors: all smd ceramic caps dielectric X5R or X7R or better\nMosfet output connectors are V+ and GND. Q1 is bed mosfet to keep high current trace short. \nSolder a thick copper wire from input to Q1 and back (both on V+ and gnd) to help with the high current.\nFor DIY purposes increase fill zones parameters."
- note added: "Output connectors are V+ and GND.\nQ1 is bed mosfet to keep high current trace short. \nSolder a thick copper wire from input to Q1 and back."
- note added: "Seems most LPC pins are 5v tolerant.\nDont abuse :)"
- note removed: "Capacitors: all smd ceramic caps dielectric X5R or X7R or better"
- note removed: "Output connectors are V+ and GND."
- note removed: "Seems most LPC pins are 5v tolerant."
Changed lines of the file:
@@
-EESchema Schematic File Version 2  date 5/21/2013 4:08:13 AM
+EESchema Schematic File Version 2  date 5/21/2013 6:39:09 AM
 LIBS:power
 LIBS:device
@@
 Text Notes 7950 700  0    79   ~ 0
 MOSFETS
-Text Notes 6050 2600 0    39   ~ 0
-Output connectors are V+ and GND.
+Text Notes 6100 2550 0    39   ~ 0
+Output connectors are V+ and GND.\nQ1 is bed mosfet to keep high current trace short. \nSolder a thick copper wire from input to Q1 and back.
 Text Notes 1000 3000 0    79   ~ 0
 Enstops and Thermistors
@@
 STEPPER DRIVERS
 Text Notes 600  5100 0    39   ~ 0
-Seems most LPC pins are 5v tolerant.
+Seems most LPC pins are 5v tolerant.\nDont abuse :)
 Text GLabel 3550 1750 2    30   Input ~ 0
 VIO3V3
@@
 	9900 5250 9900 5200
 Wire Notes Line
-	11300 2650 400  2650
-Wire Notes Line
-	5550 400  5550 2650
+	5550 400  5550 2700
 Wire Wire Line
 	2500 1400 2500 1100
@@
 Wire Wire Line
 	1000 6850 800  6700
-Text Notes 3600 5450 0    39   ~ 0
+Text Notes 3550 5400 0    39   ~ 0
 Pololu drivers or compatible footprint: http://www.pololu.com/catalog/category/120
-Text Notes 7450 2600 0    39   ~ 0
+Text Notes 7900 2650 0    39   ~ 0
 MOS drivers TC4452 (SOIC-8-Narrow) or TC4422A (SOIC-8-WIDE), check and adjust pcb footprint if needed.
 $Comp
@@
 	10550 1000 10850 1000
 Text Notes 3400 7350 0    39   ~ 0
-Capacitors: all smd ceramic caps dielectric X5R or X7R or better
+Capacitors: all smd ceramic caps dielectric X5R or X7R or better\nMosfet output connectors are V+ and GND. Q1 is bed mosfet to keep high current trace short. \nSolder a thick copper wire from input to Q1 and back (both on V+ and gnd) to help with the high current.\nFor DIY purposes increase fill zones parameters.
 Wire Notes Line
 	400  5500 11300 5500
@@
 	1    0    0    -1
 $EndComp
+Wire Notes Line
+	11300 2700 400  2700
 $EndSCHEMATC

Commit message: pin24 allocation
pin 24 re-allocation to enable xy
Connections:
- wire segments 419 -> 423
Changed lines of the file:
@@
-EESchema Schematic File Version 2  date 5/21/2013 6:39:09 AM
+EESchema Schematic File Version 2  date 5/23/2013 8:13:46 AM
 LIBS:power
 LIBS:device
@@
 Sheet 1 1
 Title ""
-Date "21 may 2013"
+Date "23 may 2013"
 Rev ""
 Comp ""
@@
 Connection ~ 800  7250
 Wire Wire Line
-	550  7100 1150 7100
-Wire Wire Line
 	800  7300 550  7300
 Wire Wire Line
@@
 	550  7300 550  7100
 Wire Wire Line
-	1200 7150 800  7150
-Wire Wire Line
-	1200 7200 800  7200
-Wire Wire Line
 	900  7350 800  7450
 Wire Wire Line
@@
 Wire Notes Line
 	11300 2700 400  2700
+Wire Wire Line
+	1200 7200 850  7200
+Wire Wire Line
+	850  7200 800  7250
+Wire Wire Line
+	1200 7150 850  7150
+Wire Wire Line
+	850  7150 800  7200
+Wire Wire Line
+	1150 7100 850  7100
+Wire Wire Line
+	850  7100 800  7150
+Wire Wire Line
+	550  7100 800  7100
 $EndSCHEMATC

Commit message: Fixed the logos so that they were added the proper way, with a placeholder in the schematic. Fixes #6.
Parts:
- added M1: LOGO_OSHW, OSHW_logo_large, symbol LOGO_OSHW
- added M2: LOGO_OSHW, OSHW_logo_10, symbol LOGO_OSHW
Other:
- moved on the sheet: Hole1, Hole2, Hole3, Hole4, J26, SW1, SW2
Changed lines of the file:
@@
-EESchema Schematic File Version 2  date 5/23/2013 8:13:46 AM
+EESchema Schematic File Version 2
 LIBS:power
 LIBS:device
@@
 LIBS:fet_driver
 LIBS:XpressoSmoothie-cache
-EELAYER 27 0
+EELAYER 24 0
 EELAYER END
 $Descr A4 11693 8268
@@
 L GND #PWR03
 U 1 1 51925E12
-P 7900 6900
-F 0 "#PWR03" H 7900 6900 30  0001 C CNN
-F 1 "GND" H 7900 6830 30  0001 C CNN
-F 2 "" H 7900 6900 60  0001 C CNN
-F 3 "" H 7900 6900 60  0001 C CNN
-	1    7900 6900
+P 7600 6900
+F 0 "#PWR03" H 7600 6900 30  0001 C CNN
+F 1 "GND" H 7600 6830 30  0001 C CNN
+F 2 "" H 7600 6900 60  0001 C CNN
+F 3 "" H 7600 6900 60  0001 C CNN
+	1    7600 6900
 	1    0    0    -1
 $EndComp
@@
 L +5V #PWR04
 U 1 1 51925E07
-P 7900 6500
-F 0 "#PWR04" H 7900 6590 20  0001 C CNN
-F 1 "+5V" H 7900 6590 30  0000 C CNN
-F 2 "" H 7900 6500 60  0001 C CNN
-F 3 "" H 7900 6500 60  0001 C CNN
-	1    7900 6500
+P 7600 6500
+F 0 "#PWR04" H 7600 6590 20  0001 C CNN
+F 1 "+5V" H 7600 6590 30  0000 C CNN
+F 2 "" H 7600 6500 60  0001 C CNN
+F 3 "" H 7600 6500 60  0001 C CNN
+	1    7600 6500
 	1    0    0    -1
 $EndComp
@@
 Text GLabel 1100 6100 0    30   Input ~ 0
 RESET
-Text GLabel 9550 6500 0    30   Input ~ 0
+Text GLabel 9150 6350 0    30   Input ~ 0
 PLAY/PAUSE
-Text GLabel 9500 6150 0    30   Input ~ 0
+Text GLabel 9100 6000 0    30   Input ~ 0
 RESET
 $Comp
 L GND #PWR07
 U 1 1 518FF959
-P 10400 6750
-F 0 "#PWR07" H 10400 6750 30  0001 C CNN
-F 1 "GND" H 10400 6680 30  0001 C CNN
-F 2 "" H 10400 6750 60  0001 C CNN
-F 3 "" H 10400 6750 60  0001 C CNN
-	1    10400 6750
+P 10000 6600
+F 0 "#PWR07" H 10000 6600 30  0001 C CNN
+F 1 "GND" H 10000 6530 30  0001 C CNN
+F 2 "" H 10000 6600 60  0001 C CNN
+F 3 "" H 10000 6600 60  0001 C CNN
+	1    10000 6600
 	1    0    0    -1
 $EndComp
@@
 L SW_PUSH SW2
 U 1 1 518FF94F
-P 10000 6500
-F 0 "SW2" H 10150 6610 50  0000 C CNN
-F 1 "SW_PUSH" H 10000 6420 50  0000 C CNN
-F 2 "" H 10000 6500 60  0001 C CNN
-F 3 "" H 10000 6500 60  0001 C CNN
-	1    10000 6500
+P 9600 6350
+F 0 "SW2" H 9750 6460 50  0000 C CNN
+F 1 "SW_PUSH" H 9600 6270 50  0000 C CNN
+F 2 "" H 9600 6350 60  0001 C CNN
+F 3 "" H 9600 6350 60  0001 C CNN
+	1    9600 6350
 	1    0    0    -1
 $EndComp
@@
 L SW_PUSH SW1
 U 1 1 518FF94A
-P 10000 6150
-F 0 "SW1" H 10150 6260 50  0000 C CNN
-F 1 "SW_PUSH" H 10000 6070 50  0000 C CNN
-F 2 "" H 10000 6150 60  0001 C CNN
-F 3 "" H 10000 6150 60  0001 C CNN
-	1    10000 6150
+P 9600 6000
+F 0 "SW1" H 9750 6110 50  0000 C CNN
+F 1 "SW_PUSH" H 9600 5920 50  0000 C CNN
+F 2 "" H 9600 6000 60  0001 C CNN
+F 3 "" H 9600 6000 60  0001 C CNN
+	1    9600 6000
 	1    0    0    -1
 $EndComp
@@
 Text GLabel 4100 6450 0    60   Input ~ 0
 MISO
-Text GLabel 8750 6750 2    30   Input ~ 0
+Text GLabel 8450 6750 2    30   Input ~ 0
 USB-D-
-Text GLabel 8750 6600 2    30   Input ~ 0
+Text GLabel 8450 6600 2    30   Input ~ 0
 USB-D+
 Text GLabel 2450 6400 2    30   Input ~ 0
@@
 L GND #PWR037
 U 1 1 51983269
-P 8650 6900
-F 0 "#PWR037" H 8650 6900 30  0001 C CNN
-F 1 "GND" H 8650 6830 30  0001 C CNN
-F 2 "" H 8650 6900 60  0001 C CNN
-F 3 "" H 8650 6900 60  0001 C CNN
-	1    8650 6900
+P 8350 6900
+F 0 "#PWR037" H 8350 6900 30  0001 C CNN
+F 1 "GND" H 8350 6830 30  0001 C CNN
+F 2 "" H 8350 6900 60  0001 C CNN
+F 3 "" H 8350 6900 60  0001 C CNN
+	1    8350 6900
 	1    0    0    -1
 $EndComp
@@
 L USB J26
 U 1 1 5197E8F8
-P 8300 6400
-F 0 "J26" H 8250 6800 60  0000 C CNN
-F 1 "USB" V 8050 6550 60  0000 C CNN
-F 2 "" H 8300 6400 60  0000 C CNN
-F 3 "" H 8300 6400 60  0000 C CNN
-	1    8300 6400
+P 8000 6400
+F 0 "J26" H 7950 6800 60  0000 C CNN
+F 1 "USB" V 7750 6550 60  0000 C CNN
+F 2 "" H 8000 6400 60  0000 C CNN
+F 3 "" H 8000 6400 60  0000 C CNN
+	1    8000 6400
 	1    0    0    -1
 $EndComp
@@
 L CONN_1 Hole1
 U 1 1 5197EDF9
-P 10850 6150
-F 0 "Hole1" H 10930 6150 40  0000 L CNN
-F 1 "CONN_1" H 10850 6205 30  0001 C CNN
-F 2 "" H 10850 6150 60  0000 C CNN
-F 3 "" H 10850 6150 60  0000 C CNN
-	1    10850 6150
+P 10500 6000
+F 0 "Hole1" H 10580 6000 40  0000 L CNN
+F 1 "CONN_1" H 10500 6055 30  0001 C CNN
+F 2 "" H 10500 6000 60  0000 C CNN
+F 3 "" H 10500 6000 60  0000 C CNN
+	1    10500 6000
 	1    0    0    -1
 $EndComp
@@
 L CONN_1 Hole2
 U 1 1 5197EE17
-P 10850 6250
-F 0 "Hole2" H 10930 6250 40  0000 L CNN
-F 1 "CONN_1" H 10850 6305 30  0001 C CNN
-F 2 "" H 10850 6250 60  0000 C CNN
-F 3 "" H 10850 6250 60  0000 C CNN
-	1    10850 6250
+P 10500 6100
+F 0 "Hole2" H 10580 6100 40  0000 L CNN
+F 1 "CONN_1" H 10500 6155 30  0001 C CNN
+F 2 "" H 10500 6100 60  0000 C CNN
+F 3 "" H 10500 6100 60  0000 C CNN
+	1    10500 6100
 	1    0    0    -1
 $EndComp
@@
 L CONN_1 Hole3
 U 1 1 5197EE1D
-P 10850 6350
-F 0 "Hole3" H 10930 6350 40  0000 L CNN
-F 1 "CONN_1" H 10850 6405 30  0001 C CNN
-F 2 "" H 10850 6350 60  0000 C CNN
-F 3 "" H 10850 6350 60  0000 C CNN
-	1    10850 6350
+P 10500 6200
+F 0 "Hole3" H 10580 6200 40  0000 L CNN
+F 1 "CONN_1" H 10500 6255 30  0001 C CNN
+F 2 "" H 10500 6200 60  0000 C CNN
+F 3 "" H 10500 6200 60  0000 C CNN
+	1    10500 6200
 	1    0    0    -1
 $EndComp
@@
 L CONN_1 Hole4
 U 1 1 5197EE23
-P 10850 6450
-F 0 "Hole4" H 10930 6450 40  0000 L CNN
-F 1 "CONN_1" H 10850 6505 30  0001 C CNN
-F 2 "" H 10850 6450 60  0000 C CNN
-F 3 "" H 10850 6450 60  0000 C CNN
-	1    10850 6450
+P 10500 6300
+F 0 "Hole4" H 10580 6300 40  0000 L CNN
+F 1 "CONN_1" H 10500 6355 30  0001 C CNN
+F 2 "" H 10500 6300 60  0000 C CNN
+F 3 "" H 10500 6300 60  0000 C CNN
+	1    10500 6300
 	1    0    0    -1
 $EndComp
-NoConn ~ 10700 6150
-NoConn ~ 10700 6250
-NoConn ~ 10700 6350
-NoConn ~ 10700 6450
+NoConn ~ 10350 6000
+NoConn ~ 10350 6100
+NoConn ~ 10350 6200
+NoConn ~ 10350 6300
 $Comp
 L CONN_2 Th2
@@
 Text Notes 5550 5800 0    79   ~ 0
 Expansion
-Text Notes 8150 5800 0    79   ~ 0
+Text Notes 7850 5800 0    79   ~ 0
 USB
 Text Notes 9800 5800 0    79   ~ 0
@@
 	4100 6450 4150 6450
 Wire Wire Line
-	8650 6900 8650 6850
+	8350 6900 8350 6850
 Wire Wire Line
-	8650 6600 8750 6600
+	8350 6600 8450 6600
 Wire Wire Line
-	10400 6150 10400 6750
+	10000 6000 10000 6600
 Wire Wire Line
 	1100 6100 1150 6100
 Wire Wire Line
-	9550 6500 9700 6500
+	9150 6350 9300 6350
 Wire Wire Line
-	10400 6150 10300 6150
+	10000 6000 9900 6000
 Wire Wire Line
 	1150 6200 1100 6200
@@
 	1150 6250 1200 6250
 Wire Wire Line
-	10300 6500 10400 6500
-Connection ~ 10400 6500
+	9900 6350 10000 6350
+Connection ~ 10000 6350
 Wire Wire Line
-	9700 6150 9500 6150
+	9300 6000 9100 6000
 Wire Wire Line
 	2450 7300 2400 7300
@@
 	1000 3400 900  3400
 Wire Wire Line
-	8750 6750 8650 6750
+	8450 6750 8350 6750
 Wire Wire Line
 	4100 6150 4150 6150
@@
 	1450 4050 1550 4050
 Wire Wire Line
-	7900 6750 7900 6900
-Connection ~ 7900 6850
+	7600 6750 7600 6900
+Connection ~ 7600 6850
 Wire Wire Line
 	10000 750  10000 1450
@@
 	10550 1450 10550 2300
 Wire Wire Line
-	7900 6600 7900 6500
+	7600 6600 7600 6500
 Wire Wire Line
 	4800 6900 4800 7000
@@
 Wire Wire Line
 	550  7100 800  7100
+$Comp
+L LOGO_OSHW M2
+U 1 1 519E49E2
+P 9350 6900
+F 0 "M2" H 9350 7050 60  0000 C CNN
+F 1 "LOGO_OSHW" H 9350 6800 60  0000 C CNN
+F 2 "OSHW_logo_10" H 9250 6950 60  0000 C CNN
+F 3 "~" H 9350 6900 60  0000 C CNN
+	1    9350 6900
+	1    0    0    -1
+$EndComp
+$Comp
+L LOGO_OSHW M1
+U 1 1 519E49F1
+P 10550 6850
+F 0 "M1" H 10550 7000 60  0000 C CNN
+F 1 "LOGO_OSHW" H 10550 6750 60  0000 C CNN
+F 2 "OSHW_logo_large" H 10450 6900 60  0000 C CNN
+F 3 "~" H 10550 6850 60  0000 C CNN
+	1    10550 6850
+	1    0    0    -1
+$EndComp
 $EndSCHEMATC

Commit message: Hid more labels, added some in so that everything is clearly marked and there are no overlaps.
Parts:
- D10: value LED_GREEN -> V_IN
- D11: value LED_GREEN -> V_GATES
- D12: value LED_GREEN -> 3V3
- D3: value LED_RED -> POWER_1
- D4: value LED_RED -> POWER_2
- D5: value LED_RED -> POWER_3
- D6: value LED_RED -> POWER_4
Changed lines of the file:
@@
 P 10350 1600
 F 0 "D6" H 10350 1700 50  0000 C CNN
-F 1 "LED_RED" H 10350 1500 50  0000 C CNN
+F 1 "POWER_4" H 10350 1500 50  0000 C CNN
 F 2 "" H 10350 1600 60  0001 C CNN
 F 3 "" H 10350 1600 60  0001 C CNN
@@
 P 9000 1600
 F 0 "D5" H 9000 1700 50  0000 C CNN
-F 1 "LED_RED" H 9000 1500 50  0000 C CNN
+F 1 "POWER_3" H 9000 1500 50  0000 C CNN
 F 2 "" H 9000 1600 60  0001 C CNN
 F 3 "" H 9000 1600 60  0001 C CNN
@@
 P 7650 1600
 F 0 "D4" H 7650 1700 50  0000 C CNN
-F 1 "LED_RED" H 7650 1500 50  0000 C CNN
+F 1 "POWER_2" H 7650 1500 50  0000 C CNN
 F 2 "" H 7650 1600 60  0001 C CNN
 F 3 "" H 7650 1600 60  0001 C CNN
@@
 P 6300 1600
 F 0 "D3" H 6300 1700 50  0000 C CNN
-F 1 "LED_RED" H 6300 1500 50  0000 C CNN
+F 1 "POWER_1" H 6300 1500 50  0000 C CNN
 F 2 "" H 6300 1600 60  0001 C CNN
 F 3 "" H 6300 1600 60  0001 C CNN
@@
 P 4550 2050
 F 0 "D10" H 4550 2150 50  0000 C CNN
-F 1 "LED_GREEN" H 4550 1950 50  0000 C CNN
+F 1 "V_IN" H 4550 1950 50  0000 C CNN
 F 2 "" H 4550 2050 60  0001 C CNN
 F 3 "" H 4550 2050 60  0001 C CNN
@@
 P 4900 1500
 F 0 "D11" H 4900 1600 50  0000 C CNN
-F 1 "LED_GREEN" H 4900 1400 50  0000 C CNN
+F 1 "V_GATES" H 4900 1400 50  0000 C CNN
 F 2 "" H 4900 1500 60  0001 C CNN
 F 3 "" H 4900 1500 60  0001 C CNN
@@
 P 5200 2050
 F 0 "D12" H 5200 2150 50  0000 C CNN
-F 1 "LED_GREEN" H 5200 1950 50  0000 C CNN
+F 1 "3V3" H 5200 1950 50  0000 C CNN
 F 2 "" H 5200 2050 60  0001 C CNN
 F 3 "" H 5200 2050 60  0001 C CNN

Commit message: Updated resistor values, calculated based on http://led.linear1.org/1led.wiz. Closes #9.
Parts:
- R18, R19, R21, R23, R28, R29: value 3k3 -> 560
- R30: value 3k3 -> 56
Changed lines of the file:
@@
 P 10350 1100
 F 0 "R18" V 10430 1100 50  0000 C CNN
-F 1 "3k3" V 10350 1100 50  0000 C CNN
+F 1 "560" V 10350 1100 50  0000 C CNN
 F 2 "" H 10350 1100 60  0001 C CNN
 F 3 "" H 10350 1100 60  0001 C CNN
@@
 P 9000 1100
 F 0 "R23" V 9080 1100 50  0000 C CNN
-F 1 "3k3" V 9000 1100 50  0000 C CNN
+F 1 "560" V 9000 1100 50  0000 C CNN
 F 2 "" H 9000 1100 60  0001 C CNN
 F 3 "" H 9000 1100 60  0001 C CNN
@@
 P 7650 1100
 F 0 "R21" V 7730 1100 50  0000 C CNN
-F 1 "3k3" V 7650 1100 50  0000 C CNN
+F 1 "560" V 7650 1100 50  0000 C CNN
 F 2 "" H 7650 1100 60  0001 C CNN
 F 3 "" H 7650 1100 60  0001 C CNN
@@
 P 6300 1100
 F 0 "R19" V 6380 1100 50  0000 C CNN
-F 1 "3k3" V 6300 1100 50  0000 C CNN
+F 1 "560" V 6300 1100 50  0000 C CNN
 F 2 "" H 6300 1100 60  0001 C CNN
 F 3 "" H 6300 1100 60  0001 C CNN
@@
 P 4550 1550
 F 0 "R28" V 4630 1550 50  0000 C CNN
-F 1 "3k3" V 4550 1550 50  0000 C CNN
+F 1 "560" V 4550 1550 50  0000 C CNN
 F 2 "" H 4550 1550 60  0001 C CNN
 F 3 "" H 4550 1550 60  0001 C CNN
@@
 P 4900 2000
 F 0 "R29" V 4980 2000 50  0000 C CNN
-F 1 "3k3" V 4900 2000 50  0000 C CNN
+F 1 "560" V 4900 2000 50  0000 C CNN
 F 2 "" H 4900 2000 60  0001 C CNN
 F 3 "" H 4900 2000 60  0001 C CNN
@@
 P 5200 1550
 F 0 "R30" V 5280 1550 50  0000 C CNN
-F 1 "3k3" V 5200 1550 50  0000 C CNN
+F 1 "56" V 5200 1550 50  0000 C CNN
 F 2 "" H 5200 1550 60  0001 C CNN
 F 3 "" H 5200 1550 60  0001 C CNN
