File: XpressoSmoothie.sch (KiCad schematic (older format))
At the start: 116 parts, among them J1 HEADER_4, J10 HEADER_3X2, J11 Pwr_in, J12 HEADER_4, J13 HEADER_4, J14 HEADER_3X2, J15 HEADER_4, J16 HEADER_3, J17 HEADER_3, J18 HEADER_3, J19 HEADER_2, J2 HEADER_4, J20 HEADER_2, J21 HEADER_2, J22 HEADER_2, J23 HEADER_3, J24 HEADER_3, J25 HEADER_3, J26 USB, J27 HEADER_4, J3 HEADER_3, J4 HEADER_3X2, J5 HEADER_3X2, J6 LPCXPRESSO_GENERIC_HEADER, J7 HEADER_4, J8 HEADER_4, J9 HEADER_3X2, M1 LOGO_OSHW, M2 LOGO_OSHW, Q1 IRLB 8743, Q2 IRLB 8743, Q3 IRLB 8743, Q4 IRLB 8743, SW1 SW_PUSH, SW2 SW_PUSH, U1 POLOLU_A4988, U10 TC4422A, U11 TC4422A, U12 LM1117-3.3, U2 POLOLU_A4988, U3 POLOLU_A4988, U4 POLOLU_A4988, U5 POLOLU_A4988, U6 CONN_MICROSD, U7 LM7812CT, U8 TC4422A, U9 TC4422A

Commit message: Switched over to minimal Molex SD card connector.
Parts:
- removed U6: CONN_MICROSD, symbol CONN_MICROSD
- added J28: MICROSD-MOLEX, symbol MICROSD-MOLEX
Connections:
- wire segments 423 -> 419
Other:
- moved on the sheet: C22, J13, J27
Changed lines of the file:
@@
 LIBS:lm1117
 LIBS:fet_driver
+LIBS:microsd-molex
 LIBS:XpressoSmoothie-cache
 EELAYER 24 0
@@
 CS
 $Comp
-L CONN_MICROSD U6
-U 1 1 51928A47
-P 4450 6600
-F 0 "U6" H 4450 6100 40  0000 C CNN
-F 1 "CONN_MICROSD" H 4500 7150 30  0000 C CNN
-F 2 "" H 4450 6600 60  0001 C CNN
-F 3 "" H 4450 6600 60  0001 C CNN
-	1    4450 6600
-	1    0    0    -1
-$EndComp
-$Comp
 L GND #PWR03
 U 1 1 51925E12
@@
 L VCC #PWR08
 U 1 1 518FF74C
-P 3700 6500
-F 0 "#PWR08" H 3700 6600 30  0001 C CNN
-F 1 "VCC" H 3700 6600 30  0000 C CNN
-F 2 "" H 3700 6500 60  0001 C CNN
-F 3 "" H 3700 6500 60  0001 C CNN
-	1    3700 6500
+P 5450 5900
+F 0 "#PWR08" H 5450 6000 30  0001 C CNN
+F 1 "VCC" H 5450 6000 30  0000 C CNN
+F 2 "" H 5450 5900 60  0001 C CNN
+F 3 "" H 5450 5900 60  0001 C CNN
+	1    5450 5900
 	1    0    0    -1
 $EndComp
@@
 L GND #PWR09
 U 1 1 518FF740
-P 3700 7000
-F 0 "#PWR09" H 3700 7000 30  0001 C CNN
-F 1 "GND" H 3700 6930 30  0001 C CNN
-F 2 "" H 3700 7000 60  0001 C CNN
-F 3 "" H 3700 7000 60  0001 C CNN
-	1    3700 7000
+P 5450 7050
+F 0 "#PWR09" H 5450 7050 30  0001 C CNN
+F 1 "GND" H 5450 6980 30  0001 C CNN
+F 2 "" H 5450 7050 60  0001 C CNN
+F 3 "" H 5450 7050 60  0001 C CNN
+	1    5450 7050
 	1    0    0    -1
 $EndComp
-Text GLabel 4100 6150 0    60   Input ~ 0
+Text GLabel 3800 6200 0    60   Input ~ 0
 CS
-Text GLabel 4100 6900 0    60   Input ~ 0
+Text GLabel 3800 6300 0    60   Input ~ 0
 MOSI
-Text GLabel 4100 6600 0    60   Input ~ 0
+Text GLabel 3800 6450 0    60   Input ~ 0
 SCK
-Text GLabel 4100 6450 0    60   Input ~ 0
+Text GLabel 3800 6550 0    60   Input ~ 0
 MISO
 Text GLabel 8450 6750 2    30   Input ~ 0
@@
 	1    0    0    -1
 $EndComp
-Text GLabel 4100 6000 0    30   Input ~ 0
+Text GLabel 3800 6900 0    30   Input ~ 0
 SD_card_detect
 $Comp
-L GND #PWR066
-U 1 1 51991CD0
-P 4800 7000
-F 0 "#PWR066" H 4800 7000 30  0001 C CNN
-F 1 "GND" H 4800 6930 30  0001 C CNN
-F 2 "" H 4800 7000 60  0001 C CNN
-F 3 "" H 4800 7000 60  0001 C CNN
-	1    4800 7000
-	1    0    0    -1
-$EndComp
-$Comp
 L C C22
 U 1 1 51992585
-P 3700 6750
-F 0 "C22" H 3750 6850 50  0000 L CNN
-F 1 "1u" H 3750 6650 50  0000 L CNN
-F 2 "SM1206" H 3900 6750 39  0000 C CNN
-F 3 "" H 3700 6750 60  0001 C CNN
-	1    3700 6750
+P 5450 6350
+F 0 "C22" H 5500 6450 50  0000 L CNN
+F 1 "1u" H 5500 6250 50  0000 L CNN
+F 2 "SM1206" H 5650 6350 39  0000 C CNN
+F 3 "" H 5450 6350 60  0001 C CNN
+	1    5450 6350
 	-1   0    0    -1
 $EndComp
-NoConn ~ 4150 6250
-NoConn ~ 4150 6350
+NoConn ~ 4050 6100
+NoConn ~ 4050 6650
 $Comp
-L PWR_FLAG #FLG067
+L PWR_FLAG #FLG066
 U 1 1 51972912
 P 1200 1550
-F 0 "#FLG067" H 1200 1645 30  0001 C CNN
+F 0 "#FLG066" H 1200 1645 30  0001 C CNN
 F 1 "PWR_FLAG" H 1200 1730 30  0000 C CNN
 F 2 "" H 1200 1550 60  0001 C CNN
@@
 $EndComp
 $Comp
-L PWR_FLAG #FLG068
+L PWR_FLAG #FLG067
 U 1 1 5197290C
 P 1200 2050
-F 0 "#FLG068" H 1200 2145 30  0001 C CNN
+F 0 "#FLG067" H 1200 2145 30  0001 C CNN
 F 1 "PWR_FLAG" H 1200 2230 30  0000 C CNN
 F 2 "" H 1200 2050 60  0001 C CNN
@@
 VIO3V3
 $Comp
-L +5V #PWR069
+L +5V #PWR068
 U 1 1 51973565
 P 2550 2000
-F 0 "#PWR069" H 2550 2090 20  0001 C CNN
+F 0 "#PWR068" H 2550 2090 20  0001 C CNN
 F 1 "+5V" H 2550 2090 30  0000 C CNN
 F 2 "" H 2550 2000 60  0001 C CNN
@@
 $EndComp
 $Comp
-L VCC #PWR070
+L VCC #PWR069
 U 1 1 51988749
 P 7900 3000
-F 0 "#PWR070" H 7900 3100 30  0001 C CNN
+F 0 "#PWR069" H 7900 3100 30  0001 C CNN
 F 1 "VCC" H 7900 3100 30  0000 C CNN
 F 2 "" H 7900 3000 60  0001 C CNN
@@
 $EndComp
 $Comp
-L VCC #PWR071
+L VCC #PWR070
 U 1 1 51988755
 P 9450 3000
-F 0 "#PWR071" H 9450 3100 30  0001 C CNN
+F 0 "#PWR070" H 9450 3100 30  0001 C CNN
 F 1 "VCC" H 9450 3100 30  0000 C CNN
 F 2 "" H 9450 3000 60  0001 C CNN
@@
 $EndComp
 $Comp
-L VCC #PWR072
+L VCC #PWR071
 U 1 1 51988761
 P 11000 3000
-F 0 "#PWR072" H 11000 3100 30  0001 C CNN
+F 0 "#PWR071" H 11000 3100 30  0001 C CNN
 F 1 "VCC" H 11000 3100 30  0000 C CNN
 F 2 "" H 11000 3000 60  0001 C CNN
@@
 $EndComp
 $Comp
-L GND #PWR073
+L GND #PWR072
 U 1 1 519902B0
 P 4550 2300
-F 0 "#PWR073" H 4550 2300 30  0001 C CNN
+F 0 "#PWR072" H 4550 2300 30  0001 C CNN
 F 1 "GND" H 4550 2230 30  0001 C CNN
 F 2 "" H 4550 2300 60  0001 C CNN
@@
 $EndComp
 $Comp
-L GND #PWR074
+L GND #PWR073
 U 1 1 519902DC
 P 5200 2300
-F 0 "#PWR074" H 5200 2300 30  0001 C CNN
+F 0 "#PWR073" H 5200 2300 30  0001 C CNN
 F 1 "GND" H 5200 2230 30  0001 C CNN
 F 2 "" H 5200 2300 60  0001 C CNN
@@
 Vgates
 $Comp
-L VCC #PWR075
+L VCC #PWR074
 U 1 1 519904B2
 P 5200 1250
-F 0 "#PWR075" H 5200 1350 30  0001 C CNN
+F 0 "#PWR074" H 5200 1350 30  0001 C CNN
 F 1 "VCC" H 5200 1350 30  0000 C CNN
 F 2 "" H 5200 1250 60  0001 C CNN
@@
 L HEADER_4 J13
 U 1 1 51991996
-P 6100 6250
-F 0 "J13" V 6150 6000 60  0000 C CNN
-F 1 "HEADER_4" V 6250 6250 28  0000 C CNN
-F 2 "" H 6100 6250 60  0001 C CNN
-F 3 "" H 6100 6250 60  0001 C CNN
-F 4 "Expansion" V 6150 6250 39  0000 C CNN "Explanation"
-	1    6100 6250
+P 6500 6250
+F 0 "J13" V 6550 6000 60  0000 C CNN
+F 1 "HEADER_4" V 6650 6250 28  0000 C CNN
+F 2 "" H 6500 6250 60  0001 C CNN
+F 3 "" H 6500 6250 60  0001 C CNN
+F 4 "Expansion" V 6550 6250 39  0000 C CNN "Explanation"
+	1    6500 6250
 	1    0    0    1
 $EndComp
@@
 Text GLabel 2900 6550 2    30   Input ~ 0
 42_P2.0PWM
-Text GLabel 5800 6400 0    30   Input ~ 0
+Text GLabel 6200 6400 0    30   Input ~ 0
 18_P0.26AOUT
-Text GLabel 5800 6100 0    30   Input ~ 0
+Text GLabel 6200 6100 0    30   Input ~ 0
 38_P0.4CAN
-Text GLabel 5800 6200 0    30   Input ~ 0
+Text GLabel 6200 6200 0    30   Input ~ 0
 39_P0.5CAN
-Text GLabel 5800 6300 0    30   Input ~ 0
+Text GLabel 6200 6300 0    30   Input ~ 0
 42_P2.0PWM
-Text Notes 4050 5800 0    79   ~ 0
+Text Notes 4050 5750 0    79   ~ 0
 SD card
 Text Notes 6950 5800 0    79   ~ 0
 I2C
-Text Notes 5550 5800 0    79   ~ 0
+Text Notes 5950 5800 0    79   ~ 0
 Expansion
 Text Notes 7850 5800 0    79   ~ 0
@@
 L HEADER_4 J27
 U 1 1 51991D45
-P 6100 6850
-F 0 "J27" V 6150 6600 60  0000 C CNN
-F 1 "HEADER_4" V 6250 6850 28  0000 C CNN
-F 2 "" H 6100 6850 60  0001 C CNN
-F 3 "" H 6100 6850 60  0001 C CNN
-F 4 "Ethernet" V 6150 6850 39  0000 C CNN "Explanation"
-	1    6100 6850
+P 6500 6850
+F 0 "J27" V 6550 6600 60  0000 C CNN
+F 1 "HEADER_4" V 6650 6850 28  0000 C CNN
+F 2 "" H 6500 6850 60  0001 C CNN
+F 3 "" H 6500 6850 60  0001 C CNN
+F 4 "Ethernet" V 6550 6850 39  0000 C CNN "Explanation"
+	1    6500 6850
 	1    0    0    1
 $EndComp
@@
 Text GLabel 2900 6300 2    30   Input ~ 0
 35_TD+
-Text GLabel 5800 6700 0    30   Input ~ 0
+Text GLabel 6200 6700 0    30   Input ~ 0
 32_RD-
-Text GLabel 5800 6800 0    30   Input ~ 0
+Text GLabel 6200 6800 0    30   Input ~ 0
 33_RD+
-Text GLabel 5800 6900 0    30   Input ~ 0
+Text GLabel 6200 6900 0    30   Input ~ 0
 34_TD-
-Text GLabel 5800 7000 0    30   Input ~ 0
+Text GLabel 6200 7000 0    30   Input ~ 0
 35_TD+
 $Comp
@@
 	6500 1450 6500 2300
 Wire Wire Line
-	6000 7000 5800 7000
+	6400 7000 6200 7000
 Wire Wire Line
-	6000 6900 5800 6900
+	6400 6900 6200 6900
 Wire Wire Line
-	6000 6800 5800 6800
+	6400 6800 6200 6800
 Wire Wire Line
-	6000 6700 5800 6700
+	6400 6700 6200 6700
 Wire Wire Line
 	2750 6150 2900 6000
@@
 	3300 2650 3300 7850
 Wire Wire Line
-	5800 6400 6000 6400
+	6200 6400 6400 6400
 Wire Wire Line
-	5800 6300 6000 6300
+	6200 6300 6400 6300
 Wire Wire Line
-	5800 6200 6000 6200
+	6200 6200 6400 6200
 Wire Wire Line
-	5800 6100 6000 6100
+	6200 6100 6400 6100
 Wire Wire Line
 	2800 6650 2900 6550
@@
 	1100 6300 1150 6300
 Wire Wire Line
-	4100 6600 4150 6600
-Wire Wire Line
-	4100 6450 4150 6450
+	3800 6450 3850 6450
 Wire Wire Line
 	8350 6900 8350 6850
@@
 	8450 6750 8350 6750
 Wire Wire Line
-	4100 6150 4150 6150
+	3800 6200 3850 6200
 Wire Wire Line
-	4100 6900 4150 6900
+	3800 6300 3850 6300
 Wire Wire Line
 	10000 2450 10000 2250
@@
 	7600 6600 7600 6500
 Wire Wire Line
-	4800 6900 4800 7000
-Wire Wire Line
-	3700 6550 3700 6500
-Wire Wire Line
-	3700 7000 3700 6950
-Wire Wire Line
-	3800 6800 4150 6800
-Wire Wire Line
-	4150 6700 3800 6700
-Connection ~ 3700 6550
-Connection ~ 3700 6950
-Wire Wire Line
-	3700 6950 3800 6950
-Wire Wire Line
-	3800 6950 3800 6800
-Wire Wire Line
-	3800 6700 3800 6550
-Wire Wire Line
-	3800 6550 3700 6550
-Wire Wire Line
 	1200 1550 1200 1600
 Connection ~ 1200 1600
@@
 	1200 2050 1200 2100
 Wire Wire Line
-	4100 6000 4800 6000
-Wire Wire Line
-	4800 6000 4800 6550
-Wire Wire Line
 	2450 5950 2500 5950
 Wire Wire Line
@@
 Regulators have different pin numbering\nIf Vin is 12V then Vgates are 12V-2Vdroput= 10V
 $Comp
-L GNDPWR #PWR076
+L GNDPWR #PWR075
 U 1 1 519AC28E
 P 4900 2300
-F 0 "#PWR076" H 4900 2350 40  0001 C CNN
+F 0 "#PWR075" H 4900 2350 40  0001 C CNN
 F 1 "GNDPWR" H 4900 2220 40  0000 C CNN
 F 2 "" H 4900 2300 60  0001 C CNN
@@
 	1    0    0    -1
 $EndComp
+$Comp
+L MICROSD-MOLEX J28
+U 1 1 51A55C9B
+P 4600 6400
+F 0 "J28" H 4200 6900 60  0000 C CNN
+F 1 "MICROSD-MOLEX" H 4600 5750 60  0000 C CNN
+F 2 "" H 4350 6300 60  0000 C CNN
+F 3 "" H 4350 6300 60  0000 C CNN
+	1    4600 6400
+	1    0    0    -1
+$EndComp
+Wire Wire Line
+	3800 6550 3850 6550
+Wire Wire Line
+	3800 6900 3950 6900
+Wire Wire Line
+	5450 6150 5450 5900
+Wire Wire Line
+	5350 6050 5450 6050
+Connection ~ 5450 6050
+Wire Wire Line
+	5450 6550 5450 7050
+Wire Wire Line
+	5450 6650 5350 6650
+Wire Wire Line
+	5450 6750 5350 6750
+Connection ~ 5450 6650
+Connection ~ 5450 6750
+Wire Wire Line
+	5250 6900 5450 6900
+Connection ~ 5450 6900
 $EndSCHEMATC

Commit message: Fixed resistor values.
Parts:
- R18, R19, R21, R23, R28, R29: value 560 -> 3k3
- R30: value 56 -> 3k3
Changed lines of the file:
@@
 P 10350 1100
 F 0 "R18" V 10430 1100 50  0000 C CNN
-F 1 "560" V 10350 1100 50  0000 C CNN
+F 1 "3k3" V 10350 1100 50  0000 C CNN
 F 2 "" H 10350 1100 60  0001 C CNN
 F 3 "" H 10350 1100 60  0001 C CNN
@@
 P 9000 1100
 F 0 "R23" V 9080 1100 50  0000 C CNN
-F 1 "560" V 9000 1100 50  0000 C CNN
+F 1 "3k3" V 9000 1100 50  0000 C CNN
 F 2 "" H 9000 1100 60  0001 C CNN
 F 3 "" H 9000 1100 60  0001 C CNN
@@
 P 7650 1100
 F 0 "R21" V 7730 1100 50  0000 C CNN
-F 1 "560" V 7650 1100 50  0000 C CNN
+F 1 "3k3" V 7650 1100 50  0000 C CNN
 F 2 "" H 7650 1100 60  0001 C CNN
 F 3 "" H 7650 1100 60  0001 C CNN
@@
 P 6300 1100
 F 0 "R19" V 6380 1100 50  0000 C CNN
-F 1 "560" V 6300 1100 50  0000 C CNN
+F 1 "3k3" V 6300 1100 50  0000 C CNN
 F 2 "" H 6300 1100 60  0001 C CNN
 F 3 "" H 6300 1100 60  0001 C CNN
@@
 P 4550 1550
 F 0 "R28" V 4630 1550 50  0000 C CNN
-F 1 "560" V 4550 1550 50  0000 C CNN
+F 1 "3k3" V 4550 1550 50  0000 C CNN
 F 2 "" H 4550 1550 60  0001 C CNN
 F 3 "" H 4550 1550 60  0001 C CNN
@@
 P 4900 2000
 F 0 "R29" V 4980 2000 50  0000 C CNN
-F 1 "560" V 4900 2000 50  0000 C CNN
+F 1 "3k3" V 4900 2000 50  0000 C CNN
 F 2 "" H 4900 2000 60  0001 C CNN
 F 3 "" H 4900 2000 60  0001 C CNN
@@
 P 5200 1550
 F 0 "R30" V 5280 1550 50  0000 C CNN
-F 1 "56" V 5200 1550 50  0000 C CNN
+F 1 "3k3" V 5200 1550 50  0000 C CNN
 F 2 "" H 5200 1550 60  0001 C CNN
 F 3 "" H 5200 1550 60  0001 C CNN

Commit message: shifted uSD
shifted uSD holder more to the edge, changed resistor values (yet again)
Parts:
- D10, D11, D12: Explanation (none) -> green
- R28: value 3k3 -> 3k
- R29: value 3k3 -> 1k5
- R30: value 3k3 -> 150
Changed lines of the file:
@@
-EESchema Schematic File Version 2
+EESchema Schematic File Version 2  date 5/29/2013 7:48:04 AM
 LIBS:power
 LIBS:device
@@
 LIBS:microsd-molex
 LIBS:XpressoSmoothie-cache
-EELAYER 24 0
+EELAYER 27 0
 EELAYER END
 $Descr A4 11693 8268
@@
 Sheet 1 1
 Title ""
-Date "23 may 2013"
+Date "29 may 2013"
 Rev ""
 Comp ""
@@
 P 4550 1550
 F 0 "R28" V 4630 1550 50  0000 C CNN
-F 1 "3k3" V 4550 1550 50  0000 C CNN
+F 1 "3k" V 4550 1550 50  0000 C CNN
 F 2 "" H 4550 1550 60  0001 C CNN
 F 3 "" H 4550 1550 60  0001 C CNN
@@
 F 2 "" H 4550 2050 60  0001 C CNN
 F 3 "" H 4550 2050 60  0001 C CNN
+F 4 "green" H 4550 2200 39  0000 C CNN "Explanation"
 	1    4550 2050
 	0    1    1    0
@@
 P 4900 2000
 F 0 "R29" V 4980 2000 50  0000 C CNN
-F 1 "3k3" V 4900 2000 50  0000 C CNN
+F 1 "1k5" V 4900 2000 50  0000 C CNN
 F 2 "" H 4900 2000 60  0001 C CNN
 F 3 "" H 4900 2000 60  0001 C CNN
@@
 F 2 "" H 4900 1500 60  0001 C CNN
 F 3 "" H 4900 1500 60  0001 C CNN
+F 4 "green" H 4750 1600 39  0000 C CNN "Explanation"
 	1    4900 1500
 	0    1    1    0
@@
 P 5200 1550
 F 0 "R30" V 5280 1550 50  0000 C CNN
-F 1 "3k3" V 5200 1550 50  0000 C CNN
+F 1 "150" V 5200 1550 50  0000 C CNN
 F 2 "" H 5200 1550 60  0001 C CNN
 F 3 "" H 5200 1550 60  0001 C CNN
@@
 F 2 "" H 5200 2050 60  0001 C CNN
 F 3 "" H 5200 2050 60  0001 C CNN
+F 4 "green" H 5200 2200 39  0000 C CNN "Explanation"
 	1    5200 2050
 	0    1    1    0
