File: mbed_compat/XpressoSmoothie.sch (KiCad schematic (older format))
At the start: 116 parts, among them J1 HEADER_4, J10 HEADER_3X2, J11 Pwr_in, J12 HEADER_4, J13 HEADER_4, J14 HEADER_3X2, J15 HEADER_4, J16 HEADER_3, J17 HEADER_3, J18 HEADER_3, J19 HEADER_2, J2 HEADER_4, J20 HEADER_2, J21 HEADER_2, J22 HEADER_2, J23 HEADER_3, J24 HEADER_3, J25 HEADER_3, J26 USB, J27 HEADER_4, J28 MICROSD-MOLEX, J3 HEADER_3, J4 HEADER_3X2, J5 HEADER_3X2, J6 LPCXPRESSO_GENERIC_HEADER, J7 HEADER_4, J8 HEADER_4, J9 HEADER_3X2, M1 LOGO_OSHW, M2 LOGO_OSHW, Q1 IRLB 8743, Q2 IRLB 8743, Q3 IRLB 8743, Q4 IRLB 8743, SW1 SW_PUSH, SW2 SW_PUSH, U1 POLOLU_A4988, U10 TC4422A, U11 TC4422A, U12 LM1117-3.3, U2 POLOLU_A4988, U3 POLOLU_A4988, U4 POLOLU_A4988, U5 POLOLU_A4988, U7 LM7812CT, U8 TC4422A, U9 TC4422A

Commit message: pin alloc mbed compat
pin allocation for mbed compatibility
Parts:
- removed J13: HEADER_4, symbol HEADER_4
- added J13: HEADER_5, symbol HEADER_5
- added J29: HEADER_3, symbol HEADER_3
- added JP1: JUMPER-2, symbol JUMPER-2
- J15: Explanation (none) -> I2C
Connections:
- wire segments 419 -> 407
Other:
- note added: "Ethernet"
- note added: "MBED settings:\n- for endstops use expansion pins 1,2,3, with gnd\n- put jumper on JP1 common enable (xy+a-enable)\n- put jumper on J13 to have P0.26 drive mosfet 4\n"
- moved on the sheet: Hole1, Hole2, Hole3, Hole4, J15, J26, J27, M1, M2, SW1, SW2

Commit message: expansion 4gnd
plus 1 gnd pin for expansion
Parts:
- removed J29: HEADER_3, symbol HEADER_3
- added J29: HEADER_4, symbol HEADER_4
Changed lines of the file:
@@
-EESchema Schematic File Version 2  date 5/30/2013 10:33:30 PM
+EESchema Schematic File Version 2  date 5/30/2013 11:41:10 PM
 LIBS:power
 LIBS:device
@@
 Wire Wire Line
 	6200 6400 6400 6400
-$Comp
-L HEADER_3 J29
-U 1 1 51A7AB26
-P 6850 6100
-F 0 "J29" H 6850 6300 60  0000 C CNN
-F 1 "HEADER_3" V 7000 6150 28  0000 C CNN
-F 2 "" H 6850 6100 60  0001 C CNN
-F 3 "" H 6850 6100 60  0001 C CNN
-F 4 "gnd" V 6900 6100 39  0000 C CNN "Explanation"
-	1    6850 6100
-	-1   0    0    -1
-$EndComp
 Wire Wire Line
-	6950 6000 6950 6300
-Connection ~ 6950 6100
-Connection ~ 6950 6200
+	6900 6000 6900 6400
+Connection ~ 6900 6100
+Connection ~ 6900 6200
 $Comp
 L GND #PWR076
 U 1 1 51A7B1AF
-P 6950 6300
-F 0 "#PWR076" H 6950 6300 30  0001 C CNN
-F 1 "GND" H 6950 6230 30  0001 C CNN
-F 2 "" H 6950 6300 60  0001 C CNN
-F 3 "" H 6950 6300 60  0001 C CNN
-	1    6950 6300
+P 6900 6400
+F 0 "#PWR076" H 6900 6400 30  0001 C CNN
+F 1 "GND" H 6900 6330 30  0001 C CNN
+F 2 "" H 6900 6400 60  0001 C CNN
+F 3 "" H 6900 6400 60  0001 C CNN
+	1    6900 6400
 	1    0    0    -1
 $EndComp
@@
 Connection ~ 6200 6600
 Connection ~ 6200 6650
+$Comp
+L HEADER_4 J29
+U 1 1 51A7BEF0
+P 6800 6150
+F 0 "J29" H 6850 6400 60  0000 C CNN
+F 1 "HEADER_4" V 6950 6150 28  0000 C CNN
+F 2 "" H 6800 6150 60  0001 C CNN
+F 3 "" H 6800 6150 60  0001 C CNN
+F 4 "gnd" V 6850 6150 39  0000 C CNN "Explanation"
+	1    6800 6150
+	-1   0    0    -1
+$EndComp
+Connection ~ 6900 6300
 $EndSCHEMATC

Commit message: mos4 pwm fix
mos 4 pwm
Parts:
- removed J13: HEADER_5, symbol HEADER_5
- removed J29: HEADER_4, symbol HEADER_4
- added J13: HEADER_4X2, symbol HEADER_4X2
- added JP1: JUMPER-2, symbol JUMPER-2
- renumbered JP1 to JP2
Connections:
- wire segments 407 -> 412
Other:
- note added: "MBED settings:\n- for endstops use expansion pins 1,2,3, with gnd\n- put jumper on common enable (xy+a-enable)\n- put jumper on to have P0.26 drive mosfet 1 bed\n"
- note removed: "MBED settings:\n- for endstops use expansion pins 1,2,3, with gnd\n- put jumper on JP1 common enable (xy+a-enable)\n- put jumper on J13 to have P0.26 drive mosfet 4\n"
Changed lines of the file:
@@
-EESchema Schematic File Version 2  date 5/30/2013 11:41:10 PM
+EESchema Schematic File Version 2  date 5/31/2013 12:28:31 AM
 LIBS:power
 LIBS:device
@@
 Text GLabel 800  7050 0    30   Input ~ 0
 X-EN
-Text GLabel 2900 7050 2    30   Input ~ 0
-POWER4
 Text GLabel 2900 6700 2    30   Input ~ 0
-POWER3
+POWER4
 Text GLabel 2900 6750 2    30   Input ~ 0
-POWER2
+POWER3
 Text GLabel 2900 6800 2    30   Input ~ 0
+POWER2
+Text GLabel 2900 7050 2    30   Input ~ 0
 POWER1
 Text GLabel 10750 1250 1    30   Input ~ 0
@@
 Wire Wire Line
 	7350 6150 7350 6100
-Text Notes 5600 6850 0    39   ~ 0
- MBED settings:\n- for endstops use expansion pins 1,2,3, with gnd\n- put jumper on JP1 common enable (xy+a-enable)\n- put jumper on J13 to have P0.26 drive mosfet 4\n
+Text Notes 5600 6950 0    39   ~ 0
+ MBED settings:\n- for endstops use expansion pins 1,2,3, with gnd\n- put jumper on common enable (xy+a-enable)\n- put jumper on to have P0.26 drive mosfet 1 bed\n
 Text Notes 7350 6550 0    79   ~ 0
 Ethernet
-Text GLabel 6200 6400 0    30   Input ~ 0
-POWER4
 $Comp
-L JUMPER-2 JP1
+L JUMPER-2 JP2
 U 1 1 51A7A651
-P 6400 6600
-F 0 "JP1" H 6400 6525 30  0000 C CNN
-F 1 "JUMPER-2" H 6400 6600 30  0001 C CNN
-F 2 "" H 6400 6600 60  0000 C CNN
-F 3 "" H 6400 6600 60  0000 C CNN
-F 4 "common_enanle" H 6400 6650 28  0000 C CNN "Explanation"
-	1    6400 6600
+P 6400 6750
+F 0 "JP2" H 6400 6675 30  0000 C CNN
+F 1 "JUMPER-2" H 6400 6750 30  0001 C CNN
+F 2 "" H 6400 6750 60  0000 C CNN
+F 3 "" H 6400 6750 60  0000 C CNN
+F 4 "common_enanle" H 6400 6800 28  0000 C CNN "Explanation"
+	1    6400 6750
 	1    0    0    -1
 $EndComp
-$Comp
-L HEADER_5 J13
-U 1 1 51A7A659
-P 6500 6200
-F 0 "J13" H 6500 6500 60  0000 C CNN
-F 1 "HEADER_5" V 6650 6150 28  0000 C CNN
-F 2 "" H 6500 6200 60  0000 C CNN
-F 3 "" H 6500 6200 60  0000 C CNN
-F 4 "Expansion" V 6550 6200 39  0000 C CNN "Explanation"
-	1    6500 6200
-	1    0    0    -1
-$EndComp
-Wire Wire Line
-	6200 6400 6400 6400
 Wire Wire Line
-	6900 6000 6900 6400
-Connection ~ 6900 6100
-Connection ~ 6900 6200
+	6800 6000 6800 6400
+Connection ~ 6800 6100
+Connection ~ 6800 6200
 $Comp
 L GND #PWR076
 U 1 1 51A7B1AF
-P 6900 6400
-F 0 "#PWR076" H 6900 6400 30  0001 C CNN
-F 1 "GND" H 6900 6330 30  0001 C CNN
-F 2 "" H 6900 6400 60  0001 C CNN
-F 3 "" H 6900 6400 60  0001 C CNN
-	1    6900 6400
+P 6800 6400
+F 0 "#PWR076" H 6800 6400 30  0001 C CNN
+F 1 "GND" H 6800 6330 30  0001 C CNN
+F 2 "" H 6800 6400 60  0001 C CNN
+F 3 "" H 6800 6400 60  0001 C CNN
+	1    6800 6400
 	1    0    0    -1
 $EndComp
-Text GLabel 6200 6600 0    30   Input ~ 0
+Text GLabel 6200 6750 0    30   Input ~ 0
 Y-EN
-Text GLabel 6200 6650 0    30   Input ~ 0
+Text GLabel 6200 6800 0    30   Input ~ 0
 X-EN
-Text GLabel 6600 6600 2    30   Input ~ 0
+Text GLabel 6600 6750 2    30   Input ~ 0
 A-EN
 Wire Wire Line
-	6200 6650 6200 6600
+	6200 6800 6200 6750
 Wire Wire Line
-	6200 6600 6300 6600
+	6200 6750 6300 6750
 Wire Wire Line
-	6600 6600 6500 6600
-Connection ~ 6200 6600
-Connection ~ 6200 6650
-$Comp
-L HEADER_4 J29
-U 1 1 51A7BEF0
-P 6800 6150
-F 0 "J29" H 6850 6400 60  0000 C CNN
-F 1 "HEADER_4" V 6950 6150 28  0000 C CNN
-F 2 "" H 6800 6150 60  0001 C CNN
-F 3 "" H 6800 6150 60  0001 C CNN
-F 4 "gnd" V 6850 6150 39  0000 C CNN "Explanation"
-	1    6800 6150
-	-1   0    0    -1
+	6600 6750 6500 6750
+Connection ~ 6200 6750
+Connection ~ 6200 6800
+Connection ~ 6800 6300
+Text GLabel 6600 6550 2    30   Input ~ 0
+POWER1
+$Comp
+L HEADER_4X2 J13
+U 1 1 51A7C943
+P 6550 6150
+F 0 "J13" H 6550 6400 60  0000 C CNN
+F 1 "HEADER_4X2" H 6550 5900 28  0000 C CNN
+F 2 "" H 6550 6150 60  0000 C CNN
+F 3 "" H 6550 6150 60  0000 C CNN
+F 4 "Expansion" V 6550 6150 39  0000 C CNN "Explanation"
+	1    6550 6150
+	1    0    0    -1
+$EndComp
+Wire Wire Line
+	6700 6000 6800 6000
+Wire Wire Line
+	6700 6100 6800 6100
+Wire Wire Line
+	6700 6200 6800 6200
+Wire Wire Line
+	6700 6300 6800 6300
+$Comp
+L JUMPER-2 JP1
+U 1 1 51A7D1D1
+P 6400 6550
+F 0 "JP1" H 6400 6475 30  0000 C CNN
+F 1 "JUMPER-2" H 6400 6550 30  0001 C CNN
+F 2 "" H 6400 6550 60  0000 C CNN
+F 3 "" H 6400 6550 60  0000 C CNN
+F 4 "common_enanle" H 6400 6600 28  0000 C CNN "Explanation"
+	1    6400 6550
+	1    0    0    -1
 $EndComp
-Connection ~ 6900 6300
+Wire Wire Line
+	6300 6550 6200 6550
+Wire Wire Line
+	6600 6550 6500 6550
+Text GLabel 6200 6550 0    30   Input ~ 0
+18_P0.26AOUT
 $EndSCHEMATC

Commit message: Added jumpers for powering LPCXPresso or mbed.
Parts:
- added JP3, JP4: JUMPER-2, symbol JUMPER-2
- JP1, JP2: Explanation common_enanle -> common_enable
Connections:
- net labels added: 3V3IN, 5VIN
- wire segments 412 -> 419
- no-connect marks 8 -> 7
Other:
- note added: "NOTE: LPCXpresso \nneeds 3v3 in to the \nVIO line. Mbed needs\n 4.5V-9.0V on the \nVIN line."

Commit message: Attempting to add jumpers for mbed-compatible board.
Connections:
- net labels removed: VIO3V3
- wire segments 419 -> 418
Changed lines of the file:
@@
 Text Notes 600  5100 0    39   ~ 0
 Seems most LPC pins are 5v tolerant.\nDont abuse :)
-Text GLabel 3550 1750 2    30   Input ~ 0
-VIO3V3
 Text GLabel 850  6800 0    30   Input ~ 0
 18_P0.26AOUT
@@
 	2450 7350 2450 7400
 Wire Wire Line
-	3450 1750 3550 1750
-Wire Wire Line
 	5200 1250 5200 1300

Commit message: Finished setting up jumpers and laying power traces for mbed-compatible.
Connections:
- wire segments 418 -> 419
Changed lines of the file:
@@
 Text GLabel 6200 6550 0    30   Input ~ 0
 18_P0.26AOUT
-Text GLabel 950  6000 0    30   Input ~ 0
-5VIN
 Wire Wire Line
-	1150 6000 950  6000
+	700  6000 1150 6000
 $Comp
 L JUMPER-2 JP3
@@
 L +5V #PWR2
 U 1 1 51A7E473
-P 4100 800
-F 0 "#PWR2" H 4100 890 20  0001 C CNN
-F 1 "+5V" H 4100 890 30  0000 C CNN
-F 2 "" H 4100 800 60  0000 C CNN
-F 3 "" H 4100 800 60  0000 C CNN
-	1    4100 800
+P 700 5950
+F 0 "#PWR2" H 700 6040 20  0001 C CNN
+F 1 "+5V" H 700 6040 30  0000 C CNN
+F 2 "" H 700 5950 60  0000 C CNN
+F 3 "" H 700 5950 60  0000 C CNN
+	1    700  5950
 	1    0    0    -1
 $EndComp
@@
 Wire Wire Line
 	4050 650  4050 600
+Wire Wire Line
+	700  6000 700  5950
 $EndSCHEMATC

Commit message: Oh, duh. Since the VIN pin isn't connected to anything on the Xpresso, it doesn't need a jumper. I can just put 5V on that pin for the mbed and that Xpresso won't be hurt.
Parts:
- removed JP4: JUMPER-2, symbol JUMPER-2
Connections:
- net labels removed: 5VIN
- wire segments 419 -> 416
Other:
- note added: "NOTE: LPCXpresso \nneeds 3v3 in to the \nVIO line. This pin is\nVOUT-only on mbed.\nThis jumper will power\nthe LPCXpresso"
- note removed: "NOTE: LPCXpresso \nneeds 3v3 in to the \nVIO line. Mbed needs\n 4.5V-9.0V on the \nVIN line."
Changed lines of the file:
@@
 L JUMPER-2 JP3
 U 1 1 51A7E41E
-P 4500 650
-F 0 "JP3" H 4500 575 30  0000 C CNN
-F 1 "JUMPER-2" H 4500 650 30  0001 C CNN
-F 2 "" H 4500 650 60  0000 C CNN
-F 3 "" H 4500 650 60  0000 C CNN
-F 4 "LPCXpresso power" H 4500 700 60  0000 C CNN "Explanation"
-	1    4500 650
-	1    0    0    -1
-$EndComp
-$Comp
-L JUMPER-2 JP4
-U 1 1 51A7E437
-P 4500 900
-F 0 "JP4" H 4500 825 30  0000 C CNN
-F 1 "JUMPER-2" H 4500 900 30  0001 C CNN
-F 2 "" H 4500 900 60  0000 C CNN
-F 3 "" H 4500 900 60  0000 C CNN
-F 4 "mbed power" H 4500 950 60  0000 C CNN "Explanation"
-	1    4500 900
+P 4500 750
+F 0 "JP3" H 4500 675 30  0000 C CNN
+F 1 "JUMPER-2" H 4500 750 30  0001 C CNN
+F 2 "" H 4500 750 60  0000 C CNN
+F 3 "" H 4500 750 60  0000 C CNN
+F 4 "LPCXpresso power" H 4500 800 60  0000 C CNN "Explanation"
+	1    4500 750
 	1    0    0    -1
 $EndComp
@@
 L VCC #PWR1
 U 1 1 51A7E464
-P 4050 600
-F 0 "#PWR1" H 4050 700 30  0001 C CNN
-F 1 "VCC" H 4050 700 30  0000 C CNN
-F 2 "" H 4050 600 60  0000 C CNN
-F 3 "" H 4050 600 60  0000 C CNN
-	1    4050 600
+P 4050 700
+F 0 "#PWR1" H 4050 800 30  0001 C CNN
+F 1 "VCC" H 4050 800 30  0000 C CNN
+F 2 "" H 4050 700 60  0000 C CNN
+F 3 "" H 4050 700 60  0000 C CNN
+	1    4050 700
 	1    0    0    -1
 $EndComp
@@
 	1    0    0    -1
 $EndComp
-Text GLabel 4850 650  2    30   Input ~ 0
+Text GLabel 4850 750  2    30   Input ~ 0
 3V3IN
-Text GLabel 4850 900  2    30   Input ~ 0
-5VIN
 Wire Wire Line
-	4050 650  4400 650
+	4050 750  4400 750
 Wire Wire Line
-	4600 650  4850 650
+	4600 750  4850 750
+Text Notes 5050 650  0    30   ~ 0
+NOTE: LPCXpresso \nneeds 3v3 in to the \nVIO line. This pin is\nVOUT-only on mbed.\nThis jumper will power\nthe LPCXpresso
 Wire Wire Line
-	4850 900  4600 900
-Wire Wire Line
-	4400 900  4100 900
-Wire Wire Line
-	4100 900  4100 800
-Text Notes 5050 650  0    30   ~ 0
-NOTE: LPCXpresso \nneeds 3v3 in to the \nVIO line. Mbed needs\n 4.5V-9.0V on the \nVIN line.
-Wire Wire Line
-	4050 650  4050 600
+	4050 750  4050 700
 Wire Wire Line
 	700  6000 700  5950

Commit message: latest changes
latest changes
Parts:
- added JP4, JP5: JUMPER-2, symbol JUMPER-2
- JP3: Explanation LPCXpresso power -> LPCXpresso_3V3IN
Connections:
- net labels added: VBAT, VIN, Vin_rmot
- net labels removed: Vin
- wire segments 416 -> 420
- no-connect marks 7 -> 6
Other:
- note added: "Power in: 12V to 28V\nThe two input connector voltages must\ncome from same psu (same gnd),\nthough may have different values."
- note added: "Regulators have different pin numbering\nIf Vin_r is 12V then Vgates are 12V-2Vdroput= 10V"
- note added: "Set this jumper to supply 3.3v into pin 28 (VIO).\nLPCXpresso needs 3v3 into the VIO line. This pin is VOUT on mbed."
- note added: "Set this jumper to supply 3.3v into the pin 3 (VBAT)."
- note added: "Set this jumper to supply Vgates into the pin 2 (VIN).\nThis requires U7 = LM7809 or LM7808 (VIN=4,5-9V)"
- note removed: "NOTE: LPCXpresso \nneeds 3v3 in to the \nVIO line. This pin is\nVOUT-only on mbed.\nThis jumper will power\nthe LPCXpresso"
- note removed: "Regulators have different pin numbering\nIf Vin is 12V then Vgates are 12V-2Vdroput= 10V"
- note removed: "Vin: 12V to 28V\nThe two input connector voltages must\ncome from same psu (same gnd),\nbut may have different values."
- moved on the sheet: C13, C14, C15, C16, C6, C8, D10, D11, D12, J11, J3, R28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
