File: mbed_compat/XpressoSmoothie.sch (KiCad schematic (older format))
At the start: 121 parts, among them J1 HEADER_4, J10 HEADER_3X2, J11 Pwr_in, J12 HEADER_4, J13 HEADER_4X2, J14 HEADER_3X2, J15 HEADER_4, J16 HEADER_3, J17 HEADER_3, J18 HEADER_3, J19 HEADER_2, J2 HEADER_4, J20 HEADER_2, J21 HEADER_2, J22 HEADER_2, J23 HEADER_3, J24 HEADER_3, J25 HEADER_3, J26 USB, J27 HEADER_4, J28 MICROSD-MOLEX, J3 HEADER_3, J4 HEADER_3X2, J5 HEADER_3X2, J6 LPCXPRESSO_GENERIC_HEADER, J7 HEADER_4, J8 HEADER_4, J9 HEADER_3X2, M1 LOGO_OSHW, M2 LOGO_OSHW, Q1 IRLB 8743, Q2 IRLB 8743, Q3 IRLB 8743, Q4 IRLB 8743, SW1 SW_PUSH, SW2 SW_PUSH, U1 POLOLU_A4988, U10 TC4422A, U11 TC4422A, U12 LM1117-3.3, U2 POLOLU_A4988, U3 POLOLU_A4988, U4 POLOLU_A4988, U5 POLOLU_A4988, U7 LM7812CT, U8 TC4422A, U9 TC4422A

Commit message: endstops jumper
endstops jumper
Parts:
- added JP6: JUMPER-3, symbol JUMPER-3
Connections:
- net labels added: +3.3VP, E+
- net labels removed: VCC
- wire segments 420 -> 423
Other:
- moved on the sheet: J16, J17, J18, J23, J24, J25

Commit message: endstops 4 pins
endstops 4 pins, removed jumper selector
Parts:
- removed J16, J17, J18, J23, J24, J25: HEADER_3, symbol HEADER_3
- removed JP6: JUMPER-3, symbol JUMPER-3
- added J16, J17, J18, J23, J24, J25: HEADER_4, symbol HEADER_4
- U7: value LM7812CT -> LM7809CT
Connections:
- net labels removed: E+
Other:
- note added: "Components: all smd ceramic caps dielectric X5R or X7R or better, leds: 20mA.\nMosfet output connectors are V+ and GND. Q1 is bed mosfet to keep high current trace short. \nSolder a thick copper wire from input to Q1 and back (both on V+ and gnd) to help with the high current.\nFor DIY purposes increase fill zones parameters."
- note added: "Seems most LPC pins are 5v tolerant, but dont abuse :)\n"
- note added: "Set this jumper to supply Vgates into the pin 2 (VIN).\nThis requires vgates regulator = LM7809 (VIN=4,5-9Vmax)"
- note removed: "Capacitors: all smd ceramic caps dielectric X5R or X7R or better\nMosfet output connectors are V+ and GND. Q1 is bed mosfet to keep high current trace short. \nSolder a thick copper wire from input to Q1 and back (both on V+ and gnd) to help with the high current.\nFor DIY purposes increase fill zones parameters."
- note removed: "Seems most LPC pins are 5v tolerant.\nDont abuse :)"
- note removed: "Set this jumper to supply Vgates into the pin 2 (VIN).\nThis requires U7 = LM7809 or LM7808 (VIN=4,5-9V)"
- moved on the sheet: C10, C11, C9, R10, R11, R12, Th0, Th1, Th2
