File: optoendstop/XpressoSmoothieOpto.sch (KiCad schematic (older format))
At the start: 122 parts, among them J1 HEADER_4, J10 HEADER_3X2, J11 Pwr_in, J12 HEADER_4, J13 HEADER_4X2, J14 HEADER_3X2, J15 HEADER_4, J16 HEADER_4, J17 HEADER_4, J18 HEADER_4, J19 HEADER_2, J2 HEADER_4, J20 HEADER_2, J21 HEADER_2, J22 HEADER_2, J23 HEADER_4, J24 HEADER_4, J25 HEADER_4, J26 USB, J27 HEADER_4, J28 MICROSD-MOLEX, J3 HEADER_3, J4 HEADER_3X2, J5 HEADER_3X2, J6 LPCXPRESSO_GENERIC_HEADER, J7 HEADER_4, J8 HEADER_4, J9 HEADER_3X2, M1 LOGO_OSHW, M2 LOGO_OSHW, Q1 IRLB 8743, Q2 IRLB 8743, Q3 IRLB 8743, Q4 IRLB 8743, SW1 SW_PUSH, SW2 SW_PUSH, U1 POLOLU_A4988, U10 TC4422A, U11 TC4422A, U12 LM1117-3.3, U2 POLOLU_A4988, U3 POLOLU_A4988, U4 POLOLU_A4988, U5 POLOLU_A4988, U7 LM7809CT, U8 TC4422A, U9 TC4422A

Commit message: endstops_mod
Parts:
- added RL_diode?: 100, symbol R
- added Rp_rcv?: 1k5, symbol R
- added U?: TCST1103/2103, symbol OPTO-TRANSISTOR4
Connections:
- net labels added: Signal
- wire segments 427 -> 433
Other:
- note added: "Other optos and voltages:\nRL_diode=(VCC-VF)/IF\nRp_rcv=(VCC-VCEsat)/(IC(on)*50%)"
- moved on the sheet: J?
Changed lines of the file:
@@
-EESchema Schematic File Version 2  date 6/1/2013 8:39:24 AM
+EESchema Schematic File Version 2  date 6/1/2013 11:12:43 AM
 LIBS:power
 LIBS:device
@@
 	1    0    0    -1
 $EndComp
-Wire Notes Line
-	-1000 3450 -1050 3450
-Wire Notes Line
-	-1050 3450 -1050 3350
-Wire Notes Line
-	-1000 3350 -1100 3350
-Wire Notes Line
-	-1100 3350 -1050 3300
-Wire Notes Line
-	-1050 3300 -1000 3350
-Wire Notes Line
-	-1200 3350 -1150 3350
-Wire Notes Line
-	-1200 3150 -1200 3350
-Wire Notes Line
-	-1150 3150 -1200 3150
-Wire Notes Line
-	-1100 3200 -1150 3150
-Wire Notes Line
-	-1050 3200 -1100 3200
-Wire Notes Line
-	-1000 3150 -1050 3200
-Wire Notes Line
-	-1000 3150 -1050 3150
-Wire Notes Line
-	-1050 3150 -1000 3200
-Wire Notes Line
-	-1000 3200 -1000 3150
-Wire Notes Line
-	-1050 3250 -1000 3250
-Wire Notes Line
-	-1050 3300 -1050 3250
-Wire Notes Line
-	-1100 3250 -1150 3200
-Wire Notes Line
-	-1100 3300 -1150 3250
 Wire Wire Line
 	1950 12850 2050 12850
@@
 L HEADER_4 J?
 U 1 1 51A99107
-P 1650 1200
-F 0 "J?" H 1700 1450 60  0000 C CNN
-F 1 "HEADER_4" V 1800 1200 28  0001 C CNN
-F 2 "" H 1650 1200 60  0001 C CNN
-F 3 "" H 1650 1200 60  0001 C CNN
-F 4 "endstop" V 1700 1200 39  0000 C CNN "Explanation"
-	1    1650 1200
+P 1150 1400
+F 0 "J?" H 1200 1650 60  0000 C CNN
+F 1 "HEADER_4" V 1300 1400 28  0001 C CNN
+F 2 "" H 1150 1400 60  0001 C CNN
+F 3 "" H 1150 1400 60  0001 C CNN
+F 4 "endstop" V 1200 1400 39  0000 C CNN "Explanation"
+	1    1150 1400
 	-1   0    0    -1
 $EndComp
@@
 L GND #PWR?
 U 1 1 51A9910D
-P 1850 1150
-F 0 "#PWR?" H 1850 1150 30  0001 C CNN
-F 1 "GND" H 1850 1080 30  0001 C CNN
-F 2 "" H 1850 1150 60  0001 C CNN
-F 3 "" H 1850 1150 60  0001 C CNN
-	1    1850 1150
+P 1350 1350
+F 0 "#PWR?" H 1350 1350 30  0001 C CNN
+F 1 "GND" H 1350 1280 30  0001 C CNN
+F 2 "" H 1350 1350 60  0001 C CNN
+F 3 "" H 1350 1350 60  0001 C CNN
+	1    1350 1350
 	1    0    0    -1
 $EndComp
-Text GLabel 1900 1050 2    30   Input ~ 0
-XMIN
+Text GLabel 1400 1250 2    30   Input ~ 0
+Signal
 Wire Wire Line
-	1750 1250 1950 1250
+	1250 1450 1450 1450
 Wire Wire Line
-	1750 1350 2000 1350
+	1250 1550 1500 1550
 Wire Wire Line
-	1750 1050 1900 1050
+	1250 1250 1400 1250
 Wire Wire Line
-	1750 1150 1850 1150
+	1250 1350 1350 1350
 $Comp
 L +5V #PWR?
 U 1 1 51A99118
-P 1950 1250
-F 0 "#PWR?" H 1950 1340 20  0001 C CNN
-F 1 "+5V" H 1950 1340 30  0000 C CNN
-F 2 "" H 1950 1250 60  0000 C CNN
-F 3 "" H 1950 1250 60  0000 C CNN
-	1    1950 1250
+P 1450 1450
+F 0 "#PWR?" H 1450 1540 20  0001 C CNN
+F 1 "+5V" H 1450 1540 30  0000 C CNN
+F 2 "" H 1450 1450 60  0000 C CNN
+F 3 "" H 1450 1450 60  0000 C CNN
+	1    1450 1450
 	1    0    0    -1
 $EndComp
@@
 L +3.3VP #PWR?
 U 1 1 51A9911E
-P 2000 1350
-F 0 "#PWR?" H 2050 1380 20  0001 C CNN
-F 1 "+3.3VP" H 2000 1440 30  0000 C CNN
-F 2 "" H 2000 1350 60  0000 C CNN
-F 3 "" H 2000 1350 60  0000 C CNN
-	1    2000 1350
+P 1500 1550
+F 0 "#PWR?" H 1550 1580 20  0001 C CNN
+F 1 "+3.3VP" H 1500 1640 30  0000 C CNN
+F 2 "" H 1500 1550 60  0000 C CNN
+F 3 "" H 1500 1550 60  0000 C CNN
+	1    1500 1550
+	1    0    0    -1
+$EndComp
+$Comp
+L OPTO-TRANSISTOR4 U?
+U 1 1 51A99755
+P 3050 1500
+F 0 "U?" H 3250 1750 60  0000 C CNN
+F 1 "TCST1103/2103" H 3050 1250 39  0000 C CNN
+F 2 "" H 3050 1500 60  0000 C CNN
+F 3 "" H 3050 1500 60  0000 C CNN
+	1    3050 1500
+	1    0    0    -1
+$EndComp
+$Comp
+L +3.3VP #PWR?
+U 1 1 51A99762
+P 3000 800
+F 0 "#PWR?" H 3050 830 20  0001 C CNN
+F 1 "+3.3VP" H 3000 890 30  0000 C CNN
+F 2 "" H 3000 800 60  0000 C CNN
+F 3 "" H 3000 800 60  0000 C CNN
+	1    3000 800
+	1    0    0    -1
+$EndComp
+$Comp
+L R RL_diode?
+U 1 1 51A99778
+P 2400 1050
+F 0 "RL_diode?" V 2480 1050 50  0000 C CNN
+F 1 "100" V 2400 1050 50  0000 C CNN
+F 2 "" H 2400 1050 60  0001 C CNN
+F 3 "" H 2400 1050 60  0001 C CNN
+	1    2400 1050
+	-1   0    0    1
+$EndComp
+$Comp
+L R Rp_rcv?
+U 1 1 51A99788
+P 3650 1050
+F 0 "Rp_rcv?" V 3730 1050 50  0000 C CNN
+F 1 "1k5" V 3650 1050 50  0000 C CNN
+F 2 "" H 3650 1050 60  0001 C CNN
+F 3 "" H 3650 1050 60  0001 C CNN
+	1    3650 1050
 	1    0    0    -1
 $EndComp
+Text Notes 2350 2050 0    39   ~ 0
+Other optos and voltages:\nRL_diode=(VCC-VF)/IF\nRp_rcv=(VCC-VCEsat)/(IC(on)*50%)
+$Comp
+L GND #PWR?
+U 1 1 51A9AF11
+P 2400 1750
+F 0 "#PWR?" H 2400 1750 30  0001 C CNN
+F 1 "GND" H 2400 1680 30  0001 C CNN
+F 2 "" H 2400 1750 60  0001 C CNN
+F 3 "" H 2400 1750 60  0001 C CNN
+	1    2400 1750
+	1    0    0    -1
+$EndComp
+Wire Wire Line
+	2400 1350 2400 1300
+Wire Wire Line
+	3650 1300 3650 1350
+Wire Wire Line
+	2400 800  3650 800
+Wire Wire Line
+	3650 1650 3650 1750
+$Comp
+L GND #PWR?
+U 1 1 51A9BBF6
+P 3650 1750
+F 0 "#PWR?" H 3650 1750 30  0001 C CNN
+F 1 "GND" H 3650 1680 30  0001 C CNN
+F 2 "" H 3650 1750 60  0001 C CNN
+F 3 "" H 3650 1750 60  0001 C CNN
+	1    3650 1750
+	1    0    0    -1
+$EndComp
+Wire Wire Line
+	2400 1650 2400 1750
+Text GLabel 3800 1350 2    30   Input ~ 0
+Signal
+Wire Wire Line
+	3650 1350 3800 1350
 $EndSCHEMATC

Commit message: optos
Parts:
- removed C1, C12, C13, C14, C2, C3, C4: 100u, symbol CP1
- removed C10, C11, C9: 10u, symbol C
- removed C15, C16, C17, C18, C19, C20, C21: 220n, symbol C
- removed C22: 1u, SM1206, symbol C
- removed C23, C24, C5, C7: 1u/50v, symbol C
- removed C6, C8: 1u/50v, SM1206, symbol C
- removed D1, D2, D7, D8: 1N4007, symbol DIODE
- removed D10: V_IN, symbol LED
- removed D11: V_GATES, symbol LED
- removed D12: 3V3, symbol LED
- removed D4: POWER_2, symbol LED
- removed D5: POWER_3, symbol LED
- removed D6: POWER_4, symbol LED
- removed F1, F2: FUSE, symbol FUSE
- removed J1, J12, J15, J16, J17, J18, J23, J24, J25, J27, J7, J8: HEADER_4, symbol HEADER_4
- removed J10, J14, J4, J5, J9: HEADER_3X2, symbol HEADER_3X2
- removed J11: Pwr_in, symbol HEADER_4
- removed J13: HEADER_4X2, symbol HEADER_4X2
- removed J19, J20, J21, J22: HEADER_2, symbol HEADER_2
- removed J26: USB, symbol USB
- removed J28: MICROSD-MOLEX, symbol MICROSD-MOLEX
- removed J3: HEADER_3, symbol HEADER_3
- removed J6: LPCXPRESSO_GENERIC_HEADER, symbol LPCXPRESSO_GENERIC_HEADER
- removed JP1, JP2, JP3, JP4, JP5: JUMPER-2, symbol JUMPER-2
- removed Q1, Q2, Q3, Q4: IRLB 8743, symbol MOSFET_N_RMC
- removed R10, R11, R12, R13, R5, R6: 4k7, symbol R
- removed R14, R4, R8, R9: 1k, symbol R
- removed R15, R16, R24, R25, R30, R7: 100, symbol R
- removed R18, R19, R21, R23, R28: 1k8, symbol R
- removed R29: 680, symbol R
- removed SW1, SW2: SW_PUSH, symbol SW_PUSH
- removed Th0, Th1, Th2: CONN_2, symbol CONN_2
- removed U1, U2, U3, U4, U5: POLOLU_A4988, symbol POLOLU_A4988
- removed U10, U11, U8, U9: TC4422A, ~, symbol TC4422A
- removed U12: LM1117-3.3, TO-220, symbol LM317AT
- removed U7: LM7809CT, TO-220, symbol LM7812CT
- added D1, D2: green, symbol LED
- added J3: HEADER_4, symbol HEADER_4
- added Q1, Q2, Q3: MOS_N, ~, symbol MOS_N
- added RL_diode2, RL_diode3: 68, symbol R
- added Rp_rcv2, Rp_rcv3: 1k5, symbol R
- added U2, U3: TCST1103/2103, symbol OPTO-TRANSISTOR4
- D3: value POWER_1 -> green; Explanation (none) -> indicator
- J2: Explanation MOTOR_OUT -> endstop
- R1, R2: value 4k7 -> 100
- R3: value 1k -> 100
- RL_diode1: renamed from RL_diode?; value 100 -> 68
- gave numbers to parts that had none: 3
Connections:
- net labels added: 3V3_1, 3V3_2, 3V3_3, GND_1, GND_2, GND_3, Signal1, Signal2, Signal3
- net labels removed: +3.3VP, 18_P0.26AOUT, 32_RD-, 33_RD+, 34_TD-, 35_TD+, 38_P0.4CAN, 39_P0.5CAN, 3V3IN, 42_P2.0PWM, A-DIR, A-EN, A-STEP, B-DIR, B-EN, B-STEP, CS, GND, GNDPWR, MISO, MOSI, PLAY/PAUSE, POWER1, POWER2, POWER3, POWER4, RESET, SCK, SCL, SDA, SD_card_detect, Signal, THERM0, THERM1, THERM2, USB-D+, USB-D-, VBAT, VIN, Vgates, Vin_Hi_curr, Vin_rmot, X-DIR, X-EN, X-STEP, XMAX, XMIN, Y-DIR, Y-EN, Y-STEP, YMAX, YMIN, Z-DIR, Z-EN, Z-STEP, ZMAX, ZMIN
- wire segments 433 -> 51
- no-connect marks 6 -> 4
Other:
- note added: "3.3v values:\nTCST2103: RL_diode:68R Rp_rcv:1k5\nTCRT1000: RL_diode:82R Rp_rcv:10k\n\nOther optos and voltages:\nRL_diode=(VCC-VF)/IF\nRp_rcv=(VCC-VCEsat)/(IC(on)*50%)"
- note added: "Connector"
- note added: "GPL"
- note added: "Indicator"
- note added: "Opto"
- note added: "Optoendstop board for XpressoSmoothie"
- note added: "https://github.com/TopherMan/XpressoSmoothie"
- note removed: "Components: all smd ceramic caps dielectric X5R or X7R or better, leds: 20mA.\nMosfet output connectors are V+ and GND. Q1 is bed mosfet to keep high current trace short. \nSolder a thick copper wire from input to Q1 and back (both on V+ and gnd) to help with the high current.\nFor DIY purposes increase fill zones parameters."
- note removed: "Enstops and Thermistors"
- note removed: "Ethernet"
- note removed: "Expansion"
- note removed: "I2C"
- note removed: "LPCXpresso 1769"
- note removed: "MBED settings:\n- for endstops use expansion pins 1,2,3, with gnd\n- put jumper on common enable (xy+a-enable)\n- put jumper on to have P0.26 drive mosfet 1 bed\n"
- note removed: "MOS drivers TC4452 (SOIC-8-Narrow) or TC4422A (SOIC-8-WIDE), check and adjust pcb footprint if needed."
- note removed: "MOSFETS"
- note removed: "Other optos and voltages:\nRL_diode=(VCC-VF)/IF\nRp_rcv=(VCC-VCEsat)/(IC(on)*50%)"
- note removed: "Output connectors are V+ and GND.\nQ1 is bed mosfet to keep high current trace short. \nSolder a thick copper wire from input to Q1 and back."
- note removed: "POWER"
- note removed: "Pololu drivers or compatible footprint: http://www.pololu.com/catalog/category/120"
- note removed: "Power in: 12V to 28V\nThe two input connector voltages must\ncome from same psu (same gnd),\nthough may have different values."
- note removed: "Regulators have different pin numbering\nIf Vin_r is 12V then Vgates are 12V-2Vdroput= 10V"
- note removed: "SD card"
- note removed: "STEPPER DRIVERS"
- note removed: "Seems most LPC pins are 5v tolerant, but dont abuse :)\n"
- note removed: "Set this jumper to supply 3.3v into pin 28 (VIO).\nLPCXpresso needs 3v3 into the VIO line. This pin is VOUT on mbed."
- note removed: "Set this jumper to supply 3.3v into the pin 3 (VBAT)."
- note removed: "Set this jumper to supply Vgates into the pin 2 (VIN).\nThis requires vgates regulator = LM7809 (VIN=4,5-9Vmax)"
- note removed: "USB"
- note removed: "Vin_Hi_curr does not have led indicator"
- moved on the sheet: Hole1, Hole2, Hole3, Hole4, J1, RL_diode1, Rp_rcv1

Commit message: opto_sch
Connections:
- wire segments 51 -> 48
Other:
- moved on the sheet: D1, D2, D3, R1, R2, R3
Changed lines of the file:
@@
-EESchema Schematic File Version 2  date 6/1/2013 3:21:41 PM
+EESchema Schematic File Version 2  date 6/1/2013 6:05:36 PM
 LIBS:power
 LIBS:device
@@
 L R R1
 U 1 1 51A9CCEC
-P 5050 2250
-F 0 "R1" V 5130 2250 50  0000 C CNN
-F 1 "100" V 5050 2250 50  0000 C CNN
-F 2 "" H 5050 2250 60  0001 C CNN
-F 3 "" H 5050 2250 60  0001 C CNN
-	1    5050 2250
-	-1   0    0    1
+P 4450 2000
+F 0 "R1" V 4530 2000 50  0000 C CNN
+F 1 "100" V 4450 2000 50  0000 C CNN
+F 2 "" H 4450 2000 60  0001 C CNN
+F 3 "" H 4450 2000 60  0001 C CNN
+	1    4450 2000
+	0    1    1    0
 $EndComp
 $Comp
 L LED D1
 U 1 1 51A9CD0F
-P 5050 2750
-F 0 "D1" H 5050 2850 50  0000 C CNN
-F 1 "green" H 5050 2650 50  0000 C CNN
-F 2 "" H 5050 2750 60  0001 C CNN
-F 3 "" H 5050 2750 60  0001 C CNN
-F 4 "indicator" H 5050 2900 39  0001 C CNN "Explanation"
-	1    5050 2750
+P 4800 2200
+F 0 "D1" H 4800 2300 50  0000 C CNN
+F 1 "green" H 4800 2100 50  0000 C CNN
+F 2 "" H 4800 2200 60  0001 C CNN
+F 3 "" H 4800 2200 60  0001 C CNN
+F 4 "indicator" H 4800 2350 39  0001 C CNN "Explanation"
+	1    4800 2200
 	0    1    1    0
 $EndComp
@@
 Wire Wire Line
 	4450 2750 4500 2750
-Wire Wire Line
-	4800 2550 5050 2550
-Wire Wire Line
-	5050 2550 5050 2500
-Connection ~ 5050 2550
 Wire Notes Line
 	450  1100 11300 1100
@@
 Connection ~ 3700 2000
 Connection ~ 1350 2100
-Wire Wire Line
-	2150 2000 5050 2000
 Wire Wire Line
 	1500 2300 1250 2300
@@
 	2150 2100 2150 2000
 Wire Wire Line
-	2150 3000 5050 3000
-Wire Wire Line
 	4800 3000 4800 2950
-Wire Wire Line
-	5050 3000 5050 2950
 Connection ~ 4800 3000
 Connection ~ 2450 3000
@@
 L R R2
 U 1 1 51AA0660
-P 5050 3750
-F 0 "R2" V 5130 3750 50  0000 C CNN
-F 1 "100" V 5050 3750 50  0000 C CNN
-F 2 "" H 5050 3750 60  0001 C CNN
-F 3 "" H 5050 3750 60  0001 C CNN
-	1    5050 3750
-	-1   0    0    1
+P 4450 3500
+F 0 "R2" V 4530 3500 50  0000 C CNN
+F 1 "100" V 4450 3500 50  0000 C CNN
+F 2 "" H 4450 3500 60  0001 C CNN
+F 3 "" H 4450 3500 60  0001 C CNN
+	1    4450 3500
+	0    1    1    0
 $EndComp
 $Comp
 L LED D2
 U 1 1 51AA0667
-P 5050 4250
-F 0 "D2" H 5050 4350 50  0000 C CNN
-F 1 "green" H 5050 4150 50  0000 C CNN
-F 2 "" H 5050 4250 60  0001 C CNN
-F 3 "" H 5050 4250 60  0001 C CNN
-F 4 "indicator" H 5050 4400 39  0001 C CNN "Explanation"
-	1    5050 4250
+P 4800 3700
+F 0 "D2" H 4800 3800 50  0000 C CNN
+F 1 "green" H 4800 3600 50  0000 C CNN
+F 2 "" H 4800 3700 60  0001 C CNN
+F 3 "" H 4800 3700 60  0001 C CNN
+F 4 "indicator" H 4800 3850 39  0001 C CNN "Explanation"
+	1    4800 3700
 	0    1    1    0
 $EndComp
@@
 Wire Wire Line
 	4450 4250 4500 4250
-Wire Wire Line
-	4800 4050 5050 4050
-Wire Wire Line
-	5050 4050 5050 4000
-Connection ~ 5050 4050
 Wire Wire Line
 	1250 3700 1500 3700
@@
 Connection ~ 3700 3500
 Connection ~ 1350 3600
-Wire Wire Line
-	2150 3500 5050 3500
 Wire Wire Line
 	1500 3800 1250 3800
@@
 	2150 3600 2150 3500
 Wire Wire Line
-	2150 4500 5050 4500
-Wire Wire Line
 	4800 4500 4800 4450
-Wire Wire Line
-	5050 4500 5050 4450
 Connection ~ 4800 4500
 Connection ~ 2450 4500
@@
 L R R3
 U 1 1 51AA0910
-P 5050 5250
-F 0 "R3" V 5130 5250 50  0000 C CNN
-F 1 "100" V 5050 5250 50  0000 C CNN
-F 2 "" H 5050 5250 60  0001 C CNN
-F 3 "" H 5050 5250 60  0001 C CNN
-	1    5050 5250
-	-1   0    0    1
+P 4450 5000
+F 0 "R3" V 4530 5000 50  0000 C CNN
+F 1 "100" V 4450 5000 50  0000 C CNN
+F 2 "" H 4450 5000 60  0001 C CNN
+F 3 "" H 4450 5000 60  0001 C CNN
+	1    4450 5000
+	0    1    1    0
 $EndComp
 $Comp
 L LED D3
 U 1 1 51AA0917
-P 5050 5750
-F 0 "D3" H 5050 5850 50  0000 C CNN
-F 1 "green" H 5050 5650 50  0000 C CNN
-F 2 "" H 5050 5750 60  0001 C CNN
-F 3 "" H 5050 5750 60  0001 C CNN
-F 4 "indicator" H 5050 5900 39  0001 C CNN "Explanation"
-	1    5050 5750
+P 4800 5200
+F 0 "D3" H 4800 5300 50  0000 C CNN
+F 1 "green" H 4800 5100 50  0000 C CNN
+F 2 "" H 4800 5200 60  0001 C CNN
+F 3 "" H 4800 5200 60  0001 C CNN
+F 4 "indicator" H 4800 5350 39  0001 C CNN "Explanation"
+	1    4800 5200
 	0    1    1    0
 $EndComp
@@
 Wire Wire Line
 	4450 5750 4500 5750
-Wire Wire Line
-	4800 5550 5050 5550
-Wire Wire Line
-	5050 5550 5050 5500
-Connection ~ 5050 5550
 Wire Wire Line
 	1250 5200 1500 5200
@@
 Connection ~ 3700 5000
 Connection ~ 1350 5100
-Wire Wire Line
-	2150 5000 5050 5000
 Wire Wire Line
 	1500 5300 1250 5300
@@
 	2150 5100 2150 5000
 Wire Wire Line
-	2150 6000 5050 6000
-Wire Wire Line
 	4800 6000 4800 5950
-Wire Wire Line
-	5050 6000 5050 5950
 Connection ~ 4800 6000
 Connection ~ 2450 6000
@@
 	3700 5850 3700 6000
 Connection ~ 3700 6000
+Wire Wire Line
+	2150 3000 4800 3000
+Wire Wire Line
+	4800 2550 4800 2400
+Wire Wire Line
+	4800 2000 4700 2000
+Wire Wire Line
+	2150 2000 4200 2000
+Wire Wire Line
+	4700 3500 4800 3500
+Wire Wire Line
+	2150 3500 4200 3500
+Wire Wire Line
+	4800 4050 4800 3900
+Wire Wire Line
+	4800 4500 2150 4500
+Wire Wire Line
+	4800 5000 4700 5000
+Wire Wire Line
+	4800 5400 4800 5550
+Wire Wire Line
+	2150 5000 4200 5000
+Wire Wire Line
+	4800 6000 2150 6000
 $EndSCHEMATC

Commit message: opto-dir
opto-dir
Parts:
- added Hole? (x8): CONN_1, symbol CONN_1
Connections:
- no-connect marks 4 -> 12
Other:
- moved on the sheet: Hole1, Hole2, Hole3, Hole4
Changed lines of the file:
@@
-EESchema Schematic File Version 2  date 6/1/2013 6:05:36 PM
+EESchema Schematic File Version 2  date 6/2/2013 3:53:05 PM
 LIBS:power
 LIBS:device
@@
 Sheet 1 1
 Title ""
-Date "1 jun 2013"
+Date "2 jun 2013"
 Rev ""
 Comp ""
@@
 L CONN_1 Hole1
 U 1 1 5197EDF9
-P 10650 5950
-F 0 "Hole1" H 10730 5950 40  0000 L CNN
-F 1 "CONN_1" H 10650 6005 30  0001 C CNN
-F 2 "" H 10650 5950 60  0000 C CNN
-F 3 "" H 10650 5950 60  0000 C CNN
-	1    10650 5950
+P 10750 5950
+F 0 "Hole1" H 10830 5950 40  0000 L CNN
+F 1 "CONN_1" H 10750 6005 30  0001 C CNN
+F 2 "" H 10750 5950 60  0000 C CNN
+F 3 "" H 10750 5950 60  0000 C CNN
+	1    10750 5950
 	1    0    0    -1
 $EndComp
@@
 L CONN_1 Hole2
 U 1 1 5197EE17
-P 10650 6050
-F 0 "Hole2" H 10730 6050 40  0000 L CNN
-F 1 "CONN_1" H 10650 6105 30  0001 C CNN
-F 2 "" H 10650 6050 60  0000 C CNN
-F 3 "" H 10650 6050 60  0000 C CNN
-	1    10650 6050
+P 10750 6050
+F 0 "Hole2" H 10830 6050 40  0000 L CNN
+F 1 "CONN_1" H 10750 6105 30  0001 C CNN
+F 2 "" H 10750 6050 60  0000 C CNN
+F 3 "" H 10750 6050 60  0000 C CNN
+	1    10750 6050
 	1    0    0    -1
 $EndComp
@@
 L CONN_1 Hole3
 U 1 1 5197EE1D
-P 10650 6150
-F 0 "Hole3" H 10730 6150 40  0000 L CNN
-F 1 "CONN_1" H 10650 6205 30  0001 C CNN
-F 2 "" H 10650 6150 60  0000 C CNN
-F 3 "" H 10650 6150 60  0000 C CNN
-	1    10650 6150
+P 10750 6150
+F 0 "Hole3" H 10830 6150 40  0000 L CNN
+F 1 "CONN_1" H 10750 6205 30  0001 C CNN
+F 2 "" H 10750 6150 60  0000 C CNN
+F 3 "" H 10750 6150 60  0000 C CNN
+	1    10750 6150
 	1    0    0    -1
 $EndComp
@@
 L CONN_1 Hole4
 U 1 1 5197EE23
-P 10650 6250
-F 0 "Hole4" H 10730 6250 40  0000 L CNN
-F 1 "CONN_1" H 10650 6305 30  0001 C CNN
-F 2 "" H 10650 6250 60  0000 C CNN
-F 3 "" H 10650 6250 60  0000 C CNN
-	1    10650 6250
-	1    0    0    -1
-$EndComp
-NoConn ~ 10500 5950
-NoConn ~ 10500 6050
-NoConn ~ 10500 6150
-NoConn ~ 10500 6250
+P 10750 6250
+F 0 "Hole4" H 10830 6250 40  0000 L CNN
+F 1 "CONN_1" H 10750 6305 30  0001 C CNN
+F 2 "" H 10750 6250 60  0000 C CNN
+F 3 "" H 10750 6250 60  0000 C CNN
+	1    10750 6250
+	1    0    0    -1
+$EndComp
+NoConn ~ 10600 5950
+NoConn ~ 10600 6050
+NoConn ~ 10600 6150
+NoConn ~ 10600 6250
 $Comp
 L HEADER_4 J1
@@
 Wire Wire Line
 	4800 6000 2150 6000
+$Comp
+L CONN_1 Hole?
+U 1 1 51AB3EFE
+P 10200 5950
+F 0 "Hole?" H 10280 5950 40  0000 L CNN
+F 1 "CONN_1" H 10200 6005 30  0001 C CNN
+F 2 "" H 10200 5950 60  0000 C CNN
+F 3 "" H 10200 5950 60  0000 C CNN
+	1    10200 5950
+	1    0    0    -1
+$EndComp
+$Comp
+L CONN_1 Hole?
+U 1 1 51AB3F04
+P 10200 6050
+F 0 "Hole?" H 10280 6050 40  0000 L CNN
+F 1 "CONN_1" H 10200 6105 30  0001 C CNN
+F 2 "" H 10200 6050 60  0000 C CNN
+F 3 "" H 10200 6050 60  0000 C CNN
+	1    10200 6050
+	1    0    0    -1
+$EndComp
+$Comp
+L CONN_1 Hole?
+U 1 1 51AB3F0A
+P 10200 6150
+F 0 "Hole?" H 10280 6150 40  0000 L CNN
+F 1 "CONN_1" H 10200 6205 30  0001 C CNN
+F 2 "" H 10200 6150 60  0000 C CNN
+F 3 "" H 10200 6150 60  0000 C CNN
+	1    10200 6150
+	1    0    0    -1
+$EndComp
+$Comp
+L CONN_1 Hole?
+U 1 1 51AB3F10
+P 10200 6250
+F 0 "Hole?" H 10280 6250 40  0000 L CNN
+F 1 "CONN_1" H 10200 6305 30  0001 C CNN
+F 2 "" H 10200 6250 60  0000 C CNN
+F 3 "" H 10200 6250 60  0000 C CNN
+	1    10200 6250
+	1    0    0    -1
+$EndComp
+NoConn ~ 10050 5950
+NoConn ~ 10050 6050
+NoConn ~ 10050 6150
+NoConn ~ 10050 6250
+$Comp
+L CONN_1 Hole?
+U 1 1 51AB3F1A
+P 9650 5950
+F 0 "Hole?" H 9730 5950 40  0000 L CNN
+F 1 "CONN_1" H 9650 6005 30  0001 C CNN
+F 2 "" H 9650 5950 60  0000 C CNN
+F 3 "" H 9650 5950 60  0000 C CNN
+	1    9650 5950
+	1    0    0    -1
+$EndComp
+$Comp
+L CONN_1 Hole?
+U 1 1 51AB3F20
+P 9650 6050
+F 0 "Hole?" H 9730 6050 40  0000 L CNN
+F 1 "CONN_1" H 9650 6105 30  0001 C CNN
+F 2 "" H 9650 6050 60  0000 C CNN
+F 3 "" H 9650 6050 60  0000 C CNN
+	1    9650 6050
+	1    0    0    -1
+$EndComp
+$Comp
+L CONN_1 Hole?
+U 1 1 51AB3F26
+P 9650 6150
+F 0 "Hole?" H 9730 6150 40  0000 L CNN
+F 1 "CONN_1" H 9650 6205 30  0001 C CNN
+F 2 "" H 9650 6150 60  0000 C CNN
+F 3 "" H 9650 6150 60  0000 C CNN
+	1    9650 6150
+	1    0    0    -1
+$EndComp
+$Comp
+L CONN_1 Hole?
+U 1 1 51AB3F2C
+P 9650 6250
+F 0 "Hole?" H 9730 6250 40  0000 L CNN
+F 1 "CONN_1" H 9650 6305 30  0001 C CNN
+F 2 "" H 9650 6250 60  0000 C CNN
+F 3 "" H 9650 6250 60  0000 C CNN
+	1    9650 6250
+	1    0    0    -1
+$EndComp
+NoConn ~ 9500 5950
+NoConn ~ 9500 6050
+NoConn ~ 9500 6150
+NoConn ~ 9500 6250
 $EndSCHEMATC

Commit message: opto_lib_and_mod
Parts:
- removed U1, U2, U3: TCST1103/2103, symbol OPTO-TRANSISTOR4
- added IC1, IC11, IC2, IC21, IC3, IC31: TCST1103, ~, symbol OPTO-ENDSTOP
- added JP?: JUMPER-3, symbol JUMPER-3
- added R1?: 10k, symbol R
- Q1, Q2, Q3: value MOS_N -> BS108D
- R1, R2, R3: value 100 -> 150
- gave numbers to parts that had none: 8
Connections:
- net labels removed: +5V
- wire segments 48 -> 53
- no-connect marks 12 -> 15
Other:
- note added: "Placeholders (footprints alternates)"
- note added: "TO92: BS108D, 2N7002; \nSOT23: BSS138, BSS123;\nor others with Vgs(th) <2.5V"
- moved on the sheet: D1, Hole1, Hole10, Hole11, Hole12, Hole2, Hole3, Hole4, Hole5, Hole6, Hole7, Hole8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
