File: optoendstop/XpressoSmoothieOpto.sch (KiCad schematic (older format))
At the start: 40 parts, among them IC1 TCST1103, IC11 TCST1103, IC2 TCST1103, IC21 TCST1103, IC3 TCST1103, IC31 TCST1103, J1 HEADER_4, J2 HEADER_4, J3 HEADER_4, M1 LOGO_OSHW, M2 LOGO_OSHW, Q1 BS108D, Q2 BS108D, Q3 BS108D

Commit message: oe_mod
oe_mod
Parts:
- removed JP?: JUMPER-3, symbol JUMPER-3
- removed R1?: 10k, symbol R
Connections:
- wire segments 53 -> 51
Other:
- moved on the sheet: D2, D3
Changed lines of the file:
@@
-EESchema Schematic File Version 2  date 6/3/2013 7:52:37 PM
+EESchema Schematic File Version 2  date 6/3/2013 8:58:24 PM
 LIBS:power
 LIBS:device
@@
 Text Notes 1050 6800 0    59   ~ 0
 3.3v values:\nTCST2103:	RL_diode:68R	Rp_rcv:1k5\nTCRT1000:	RL_diode:82R	Rp_rcv:10k\n\nOther optos and voltages:\nRL_diode=(VCC-VF)/IF\nRp_rcv=(VCC-VCEsat)/(IC(on)*50%)
-Text GLabel 4150 2450 1    30   Input ~ 0
+Text GLabel 4200 2550 1    30   Input ~ 0
 Signal1
 $Comp
@@
 Text Notes 10300 800  0    197  ~ 0
 GPL
-Wire Wire Line
-	2450 2550 2450 2500
-Wire Wire Line
-	3700 2500 3700 2550
-Wire Wire Line
-	2450 2850 2450 3000
-Wire Wire Line
-	3700 2550 4050 2550
-Wire Wire Line
-	4050 2750 4500 2750
-Wire Notes Line
-	450  1100 11300 1100
-Wire Wire Line
-	1250 2200 1500 2200
-Connection ~ 2450 2000
-Connection ~ 3700 2000
-Wire Wire Line
-	1500 2300 1250 2300
 Text GLabel 1500 2000 2    30   Input ~ 0
 3V3_1
 Text GLabel 1500 2200 2    30   Input ~ 0
 GND_1
-Wire Wire Line
-	1250 2000 1500 2000
 Text GLabel 2150 2000 0    30   Input ~ 0
 3V3_1
@@
 	-1   0    0    1
 $EndComp
-Wire Wire Line
-	2150 2100 2150 2000
-Wire Wire Line
-	4800 3000 4800 2950
-Connection ~ 4800 3000
-Connection ~ 2450 3000
 Text GLabel 2150 3000 0    30   Input ~ 0
 GND_1
@@
 	1    0    0    -1
 $EndComp
-Text GLabel 3800 4050 2    30   Input ~ 0
-Signal2
 $Comp
 L MOS_N Q2
@@
 	1    0    0    -1
 $EndComp
-Text GLabel 4450 4250 0    30   Input ~ 0
-Signal2
 $Comp
 L R R2
@@
 L LED D2
 U 1 1 51AA0667
-P 4800 3700
-F 0 "D2" H 4800 3800 50  0000 C CNN
-F 1 "green" H 4800 3600 50  0000 C CNN
-F 2 "" H 4800 3700 60  0001 C CNN
-F 3 "" H 4800 3700 60  0001 C CNN
-F 4 "indicator" H 4800 3850 39  0001 C CNN "Explanation"
-	1    4800 3700
+P 4800 3800
+F 0 "D2" H 4800 3900 50  0000 C CNN
+F 1 "green" H 4800 3700 50  0000 C CNN
+F 2 "" H 4800 3800 60  0001 C CNN
+F 3 "" H 4800 3800 60  0001 C CNN
+F 4 "indicator" H 4800 3950 39  0001 C CNN "Explanation"
+	1    4800 3800
 	0    1    1    0
 $EndComp
-Wire Wire Line
-	2450 4050 2450 4000
-Wire Wire Line
-	3700 4000 3700 4050
-Wire Wire Line
-	2450 4350 2450 4500
-Wire Wire Line
-	3700 4050 3800 4050
-Wire Wire Line
-	4450 4250 4500 4250
-Wire Wire Line
-	1250 3700 1500 3700
-Connection ~ 2450 3500
-Connection ~ 3700 3500
-Wire Wire Line
-	1500 3800 1250 3800
 Text GLabel 1500 3500 2    30   Input ~ 0
 3V3_2
 Text GLabel 1500 3700 2    30   Input ~ 0
 GND_2
-Wire Wire Line
-	1250 3500 1500 3500
 Text GLabel 2150 3500 0    30   Input ~ 0
 3V3_2
@@
 	-1   0    0    1
 $EndComp
-Wire Wire Line
-	2150 3600 2150 3500
-Wire Wire Line
-	4800 4500 4800 4450
-Connection ~ 4800 4500
-Connection ~ 2450 4500
 Text GLabel 2150 4500 0    30   Input ~ 0
 GND_2
-Wire Wire Line
-	3700 3000 3700 2850
-Connection ~ 3700 3000
-Wire Wire Line
-	3700 4500 3700 4350
-Connection ~ 3700 4500
 $Comp
 L HEADER_4 J3
@@
 	1    0    0    -1
 $EndComp
-Text GLabel 3800 5550 2    30   Input ~ 0
-Signal3
 $Comp
 L MOS_N Q3
@@
 	1    0    0    -1
 $EndComp
-Text GLabel 4450 5750 0    30   Input ~ 0
-Signal3
 $Comp
 L R R3
@@
 	0    1    1    0
 $EndComp
-$Comp
-L LED D3
-U 1 1 51AA0917
-P 4800 5200
-F 0 "D3" H 4800 5300 50  0000 C CNN
-F 1 "green" H 4800 5100 50  0000 C CNN
-F 2 "" H 4800 5200 60  0001 C CNN
-F 3 "" H 4800 5200 60  0001 C CNN
-F 4 "indicator" H 4800 5350 39  0001 C CNN "Explanation"
-	1    4800 5200
-	0    1    1    0
-$EndComp
-Wire Wire Line
-	2450 5550 2450 5500
-Wire Wire Line
-	3700 5500 3700 5550
-Wire Wire Line
-	2450 5850 2450 6000
-Wire Wire Line
-	3700 5550 3800 5550
-Wire Wire Line
-	4450 5750 4500 5750
-Wire Wire Line
-	1250 5200 1500 5200
-Connection ~ 2450 5000
-Connection ~ 3700 5000
-Wire Wire Line
-	1500 5300 1250 5300
 Text GLabel 1500 5000 2    30   Input ~ 0
 3V3_3
 Text GLabel 1500 5200 2    30   Input ~ 0
 GND_3
-Wire Wire Line
-	1250 5000 1500 5000
 Text GLabel 2150 5000 0    30   Input ~ 0
 3V3_3
@@
 	-1   0    0    1
 $EndComp
-Wire Wire Line
-	2150 5100 2150 5000
-Wire Wire Line
-	4800 6000 4800 5950
-Connection ~ 4800 6000
-Connection ~ 2450 6000
 Text GLabel 2150 6000 0    30   Input ~ 0
 GND_3
-Wire Wire Line
-	3700 6000 3700 5850
-Connection ~ 3700 6000
-Wire Wire Line
-	2150 3000 5000 3000
-Wire Wire Line
-	4800 2550 4800 2500
-Wire Wire Line
-	2150 2000 4200 2000
-Wire Wire Line
-	4700 3500 4800 3500
-Wire Wire Line
-	2150 3500 4200 3500
-Wire Wire Line
-	4800 4050 4800 3900
-Wire Wire Line
-	2150 4500 4800 4500
-Wire Wire Line
-	4800 5000 4700 5000
-Wire Wire Line
-	4800 5400 4800 5550
-Wire Wire Line
-	2150 5000 4200 5000
-Wire Wire Line
-	2150 6000 4800 6000
 $Comp
 L CONN_1 Hole9
@@
 Placeholders (footprints alternates)
 $Comp
-L R R1?
-U 1 1 51ACC85C
-P 5000 2550
-F 0 "R1?" V 5080 2550 50  0000 C CNN
-F 1 "10k" V 5000 2550 50  0000 C CNN
-F 2 "" H 5000 2550 60  0001 C CNN
-F 3 "" H 5000 2550 60  0001 C CNN
-	1    5000 2550
-	1    0    0    -1
-$EndComp
-Wire Wire Line
-	4700 2000 5000 2000
+L LED D3
+U 1 1 51AA0917
+P 4800 5300
+F 0 "D3" H 4800 5400 50  0000 C CNN
+F 1 "green" H 4800 5200 50  0000 C CNN
+F 2 "" H 4800 5300 60  0001 C CNN
+F 3 "" H 4800 5300 60  0001 C CNN
+F 4 "indicator" H 4800 5450 39  0001 C CNN "Explanation"
+	1    4800 5300
+	0    1    1    0
+$EndComp
+Text GLabel 4200 4050 1    30   Input ~ 0
+Signal2
+Text GLabel 4200 5550 1    30   Input ~ 0
+Signal3
+Wire Wire Line
+	2450 2550 2450 2500
+Wire Wire Line
+	3700 2500 3700 2550
+Wire Wire Line
+	2450 2850 2450 3000
+Wire Notes Line
+	450  1100 11300 1100
+Wire Wire Line
+	1250 2200 1500 2200
+Connection ~ 2450 2000
+Connection ~ 3700 2000
+Wire Wire Line
+	1500 2300 1250 2300
+Wire Wire Line
+	1250 2000 1500 2000
+Wire Wire Line
+	2150 2100 2150 2000
+Wire Wire Line
+	4800 3000 4800 2950
+Connection ~ 4800 3000
+Connection ~ 2450 3000
+Wire Wire Line
+	2450 4050 2450 4000
+Wire Wire Line
+	3700 4000 3700 4050
+Wire Wire Line
+	2450 4350 2450 4500
+Wire Wire Line
+	1250 3700 1500 3700
+Connection ~ 2450 3500
+Connection ~ 3700 3500
+Wire Wire Line
+	1500 3800 1250 3800
+Wire Wire Line
+	1250 3500 1500 3500
+Wire Wire Line
+	2150 3600 2150 3500
+Wire Wire Line
+	4800 4500 4800 4450
+Connection ~ 4800 4500
+Connection ~ 2450 4500
+Wire Wire Line
+	3700 3000 3700 2850
+Connection ~ 3700 3000
+Wire Wire Line
+	3700 4500 3700 4350
+Connection ~ 3700 4500
+Wire Wire Line
+	2450 5550 2450 5500
+Wire Wire Line
+	3700 5500 3700 5550
+Wire Wire Line
+	2450 5850 2450 6000
+Wire Wire Line
+	1250 5200 1500 5200
+Connection ~ 2450 5000
+Connection ~ 3700 5000
+Wire Wire Line
+	1500 5300 1250 5300
+Wire Wire Line
+	1250 5000 1500 5000
+Wire Wire Line
+	2150 5100 2150 5000
+Wire Wire Line
+	4800 6000 4800 5950
+Connection ~ 4800 6000
+Connection ~ 2450 6000
+Wire Wire Line
+	3700 6000 3700 5850
+Connection ~ 3700 6000
+Wire Wire Line
+	2150 3000 4800 3000
+Wire Wire Line
+	4800 2550 4800 2500
+Wire Wire Line
+	2150 2000 4200 2000
+Wire Wire Line
+	2150 3500 4200 3500
+Wire Wire Line
+	4800 4050 4800 4000
+Wire Wire Line
+	2150 4500 4800 4500
+Wire Wire Line
+	4800 5500 4800 5550
+Wire Wire Line
+	2150 5000 4200 5000
+Wire Wire Line
+	2150 6000 4800 6000
+Wire Wire Line
+	4700 2000 4800 2000
 Wire Wire Line
 	4800 2000 4800 2100
-Wire Wire Line
-	5000 2000 5000 2300
 Connection ~ 4800 2000
-Wire Wire Line
-	5000 3000 5000 2800
-$Comp
-L JUMPER-3 JP?
-U 1 1 51ACC996
-P 4150 2550
-F 0 "JP?" H 4150 2490 30  0000 C CNN
-F 1 "JUMPER-3" H 4150 2550 30  0001 C CNN
-F 2 "" H 4150 2550 60  0000 C CNN
-F 3 "" H 4150 2550 60  0000 C CNN
-	1    4150 2550
-	-1   0    0    -1
-$EndComp
-Wire Wire Line
-	4050 2550 4050 2750
 Connection ~ 4800 2100
 Wire Wire Line
-	4250 2550 4550 2550
-Wire Wire Line
-	4550 2550 4550 2100
-Wire Wire Line
-	4550 2100 4800 2100
-Wire Wire Line
-	4150 2500 4150 2450
+	4700 3500 4800 3500
+Wire Wire Line
+	4800 3500 4800 3600
+Wire Wire Line
+	4700 5000 4800 5000
+Wire Wire Line
+	4800 5000 4800 5100
+Connection ~ 4800 5000
+Connection ~ 4800 3500
+Wire Wire Line
+	3700 2550 4200 2550
+Wire Wire Line
+	3700 4050 4200 4050
+Wire Wire Line
+	4200 4050 4200 4250
+Wire Wire Line
+	4200 4250 4500 4250
+Wire Wire Line
+	4200 2550 4200 2750
+Wire Wire Line
+	4200 2750 4500 2750
+Wire Wire Line
+	4200 5750 4200 5550
+Wire Wire Line
+	4200 5550 3700 5550
+Wire Wire Line
+	4200 5750 4500 5750
 $EndSCHEMATC

Commit message: optoendstops
optoendstops
Parts:
- removed D2, D3: green, symbol LED
- removed Hole10, Hole11, Hole12, Hole5, Hole6, Hole7, Hole8, Hole9: CONN_1, symbol CONN_1
- removed IC2, IC21, IC3, IC31: TCST1103, ~, symbol OPTO-ENDSTOP
- removed J2, J3: HEADER_4, symbol HEADER_4
- removed M1: LOGO_OSHW, OSHW_logo_large, symbol LOGO_OSHW
- removed Q2, Q3: BS108D, ~, symbol MOS_N
- removed R2, R3: 150, symbol R
- removed RL_diode2, RL_diode3: 68, symbol R
- removed Rp_rcv2, Rp_rcv3: 1k5, symbol R
- added JP1: JUMPER-3, symbol JUMPER-3
Connections:
- net labels added: 3.3V, 5V, GND
- net labels removed: 3V3_1, 3V3_2, 3V3_3, GND_1, GND_2, GND_3, Signal2, Signal3
- wire segments 51 -> 22
- no-connect marks 15 -> 4
Other:
- note added: "3.3v values:\nTCST1103: RL_diode:68R Rp_rcv:1k5\nTCRT1000: RL_diode:82R Rp_rcv:10k\n\n5v values:\nTCST1103: RL_diode:120R Rp_rcv:2k2\nTCRT1000: RL_diode:150R Rp_rcv:1k5\n"
- note added: "TO92: BS108D, 2N7002; \nSOT23: BSS138, BSS123;\nor others with Vgs(th) < 2.5V"
- note added: "hardwired with 3.3v"
- note removed: "3.3v values:\nTCST2103: RL_diode:68R Rp_rcv:1k5\nTCRT1000: RL_diode:82R Rp_rcv:10k\n\nOther optos and voltages:\nRL_diode=(VCC-VF)/IF\nRp_rcv=(VCC-VCEsat)/(IC(on)*50%)"
- note removed: "Placeholders (footprints alternates)"
- note removed: "TO92: BS108D, 2N7002; \nSOT23: BSS138, BSS123;\nor others with Vgs(th) <2.5V"
- moved on the sheet: D1, Hole1, Hole2, Hole3, Hole4, IC1, IC11, M2, Q1, R1, RL_diode1, Rp_rcv1

Commit message: optod-rem-jumper
removed jumper
Parts:
- removed JP1: JUMPER-3, symbol JUMPER-3
Connections:
- wire segments 22 -> 17
Other:
- note removed: "hardwired with 3.3v"
Changed lines of the file:
@@
-EESchema Schematic File Version 2  date 6/4/2013 4:22:04 AM
+EESchema Schematic File Version 2  date 6/4/2013 4:47:08 AM
 LIBS:power
 LIBS:device
@@
 	5400 2550 5400 2500
 Wire Wire Line
-	2900 2000 4800 2000
+	2700 2000 4800 2000
 Wire Wire Line
 	5300 2000 5400 2000
@@
 Wire Wire Line
 	4800 2750 5100 2750
-$Comp
-L JUMPER-3 JP1
-U 1 1 51AD3A26
-P 2850 2100
-F 0 "JP1" H 2850 2000 30  0000 C CNN
-F 1 "JUMPER-3" H 2850 2100 30  0001 C CNN
-F 2 "" H 2850 2100 60  0000 C CNN
-F 3 "" H 2850 2100 60  0000 C CNN
-	1    2850 2100
-	0    1    -1   0
-$EndComp
-Wire Wire Line
-	2700 2000 2850 2000
-Wire Wire Line
-	2700 2200 2850 2200
-Wire Wire Line
-	2900 2100 2900 2000
 $Comp
 L PWR_FLAG #FLG01
@@
 Text GLabel 2700 2000 0    30   Input ~ 0
 3.3V
-Text GLabel 2700 2200 0    30   Input ~ 0
-5V
 Text GLabel 2700 3000 0    30   Input ~ 0
 GND
 Connection ~ 1250 2100
 Connection ~ 1250 2000
-Wire Wire Line
-	2800 2100 2900 2100
-Wire Wire Line
-	2800 2100 2800 2000
-Connection ~ 2800 2000
-Text Notes 2600 1950 0    39   ~ 0
-hardwired with 3.3v
 $EndSCHEMATC
